File: schematics/Rotor_kicad/LIOD_interface.kicad_sch (KiCad schematic)
At the start: 0 parts

Commit message: Fixed mistakes in main board schematics
Parts:
- added C37, C38: 100n, symbol Device:C
- added CN1L1: LIOD interface connector, symbol Connector_Generic:Conn_02x06_Counter_Clockwise
- added CN2L1: "Debit reader", symbol Connector_Generic:Conn_02x05_Counter_Clockwise
- added CN3L2: LIOD cable, symbol Connector_Generic:Conn_02x05_Counter_Clockwise
- added D27, D28: 1N4148, Diode_THT:D_DO-35_SOD27_P7.62mm_Horizontal, symbol Diode:1N4148
- added R100, R91: 100k?, symbol Device:R
- added R101, R113, R94, R95, R96: 100k, symbol Device:R
- added R102, R104, R105, R106, R107, R108, R109, R110, R111, R112, R97, R99: ?, symbol Device:R
- added R103, R90, R92: ~, symbol Device:R
- added R93: 47k, symbol Device:R
- added R98: 100k(?), symbol Device:R
- added SUR2: ~, symbol IPM_custom:LIOD_PSU
- added T13, T14, T15, T16, T17, T18: BC337, Package_TO_SOT_THT:TO-92_Inline, symbol Transistor_BJT:BC337
- added U19: 74HC04, symbol 74xx:74HC04
- added U20: 74HC240, symbol 74xx:74HC240
- added U21: 4017, symbol 4xxx:4017
Connections:
- new net: R110.1, T17.1 (C)
- new net: R104.1, R107.2, T17.2 (B)
- new net: R90.1, R91.1, T13.2 (B)
- new net: R96.2, T14.1 (C), U20.15 (2A1)
- new net: R102.1, R99.1, T14.2 (B)
- new net: R97.2, T15.1 (C), U20.13 (2A2)
- new net: R100.1, R103.1, T15.2 (B)
- new net: CN1L1.6 (Pin_6), SUR2.3 (UNK)
- new net: R104.2, U21.5 (Q6)
- new net: R92.2, T13.1 (C), U19.1, U21.14 (CLK)
- new net: R93.2, U19.2
- new net: C38.2, CN3L2.9 (Pin_9), D28.2 (A), R108.1
- new net: C37.1, U19.11, U19.6
- new net: C37.2, R93.1, U19.3
- new net: U19.10, U19.9, U20.1 (1OE)
- new net: R95.2, U20.11 (2A3), U20.5 (2Y1)
- new net: R94.2, U20.14 (1Y2), U20.2 (1A0)
- new net: U19.8, U20.19 (2OE)
- new net: CN3L2.3 (Pin_3), R98.1, U20.4 (1A1)
- new net: CN3L2.1 (Pin_1), R101.1, U20.6 (1A2)
- new net: U19.12, U20.8 (1A3), U21.15 (Reset)
- new net: U19.4, U19.5
- new net: CN2L1.5 (Pin_5), SUR2.5 (UNK2)
- new net: R111.1, R112.2, T18.2 (B)
- new net: R105.2, U21.9 (Q8)
- new net: CN2L1.9 (Pin_9), D27.2 (A), R110.2
- new net: CN2L1.8 (Pin_8), R109.1
- new net: CN2L1.10 (Pin_10), R109.2, T18.1 (C)
- new net: R108.2, T16.1 (C)
- new net +5V: CN1L1.8 (Pin_8), CN3L2.8 (Pin_8), R113.1, R92.1, R96.1, R97.1, U19.14 (VCC), U20.20 (VCC), U21.16 (VDD)
- new net +BATT: CN1L1.7 (Pin_7), CN3L2.5 (Pin_5), SUR2.1 (VBAT)
- new net CN1L-1: CN1L1.1 (Pin_1), U20.18 (1Y0), U20.7 (2Y2)
- new net CN1L-3: CN1L1.3 (Pin_3), U20.16 (1Y1), U20.9 (2Y3)
- new net CN1L-4: CN1L1.4 (Pin_4), D27.1 (K), D28.1 (K)
- new net CN1L-5: CN1L1.5 (Pin_5), CN2L1.2 (Pin_2), CN3L2.2 (Pin_2), R105.1, R106.1, T16.2 (B)
- new net CN2L-1: CN1L1.10 (Pin_10), CN2L1.1 (Pin_1), R103.2, R90.2
- new net CN2L-3: CN2L1.3 (Pin_3), R102.2
- new net GND: C38.1, CN1L1.11 (Pin_11), CN1L1.12 (Pin_12), CN1L1.9 (Pin_9), CN2L1.4 (Pin_4), CN2L1.7 (Pin_7), CN3L2.4 (Pin_4), CN3L2.7 (Pin_7), R100.2, R101.2, R106.2, R107.1, R111.2, R91.2, R94.1, R95.1, R98.2, R99.2, SUR2.2 (GND1), SUR2.4 (GND2), T13.3 (E), T14.3 (E), T15.3 (E), T16.3 (E), T17.3 (E), T18.3 (E), U19.7 (GND), U20.10 (GND), U21.13 (CKEN), U21.8 (VSS)
- new net LIOD_RESET: CN3L2.10 (Pin_10), U20.12 (1Y3)
- new net ~{LIOD_RESET_BUFF}: R112.1, R113.2, U20.3 (2Y0)
- new net ~{LIOD_RESET}: CN1L1.2 (Pin_2), U19.13, U20.17 (2A0)
- no-connect marks 0 -> 11
