File: schematics/Rotor_kicad/Rotor_kicad.kicad_sch (KiCad schematic)
At the start: 251 parts, among them CN1 ., CN1 LIOD interface connector, CN2 Front panel, CN2 Unknown, CN2B Front panel, CN3 Headset, CN3 LIOD cable, CN4 Battery, CN5 Coin tray, CN6 Ext safe, CN6 LIOD, J1 ., Q1 BC847, Q4 BC847, Q7 BC857, Q8 BC857, SW1 1, SW1 Left, SW10 0, SW11 #, SW2 2, SW2 Right, SW3 3, SW4 4, SW5 5, SW6 6, SW7 7, SW8 8, SW9 *, SW9 9, T1 BC327, T10 BC327, T11 BC237, T12 BC237, T2 MPSA42, T3 MPSA92, T5 MPSA42, T6 BC337, T6 MPSA42, T7 MPSA42, T8 MPSA42, T9 BU806, U1 4001, U1 40106, U1 74HC14, U1 74HC240, U1 HEF4093B, U1 LS358B, U2 74HC04, U2 ICL7665, U3 4017

Commit message: New schematics!
Parts:
- removed CN2: Unknown, symbol Connector_Generic:Conn_02x06_Counter_Clockwise
- removed CN3: LIOD cable, symbol Connector_Generic:Conn_02x05_Counter_Clockwise
- removed D2: 1N4148, Diode_THT:D_DO-35_SOD27_P7.62mm_Horizontal, symbol Diode:1N4148
- removed D4: ?, Diode_THT:D_DO-41_SOD81_P10.16mm_Horizontal, symbol Diode:1N4007
- removed J?: ., symbol Connector:Conn_01x20_Male
- removed M?: Rotor, symbol Motor:Motor_DC
- removed Q4, Q? (x2): BC847, Package_TO_SOT_SMD:SOT-23, symbol Transistor_BJT:BC847
- removed Q7, Q?: BC857, Package_TO_SOT_SMD:SOT-23, symbol Transistor_BJT:BC857
- removed Q? (x2): BCW67, Package_TO_SOT_SMD:SOT-23, symbol Transistor_BJT:BC857
- removed R? (x2): 220, symbol Device:R
- removed R? (x4): 6.5K, symbol Device:R
- removed R? (x2): 210, symbol Device:R
- removed R?: 100, symbol Device:R
- removed R?: 100K, symbol Device:R
- removed R?: 10, symbol Device:R
- removed U1: 4001, symbol 4xxx:4001
- added AR2: ~, Resistor_THT:R_Array_SIP9, symbol Device:R_Network08
- added C1 (x2), C10, C11, C12, C19, C2 (x2), C21, C22, C3, C4, C5 (x2), C6, C7, C8, C9: 100n, symbol Device:C
- added C13, C14: ~, symbol Device:C_Polarized
- added CN1: Mechanical section connector, symbol Connector_Generic:Conn_02x30_Counter_Clockwise
- added CN2: Line interface connector, symbol Connector_Generic:Conn_02x20_Counter_Clockwise
- added CN2L: "Debit reader", symbol Connector_Generic:Conn_02x05_Counter_Clockwise
- added CN3L1: LIOD cable, symbol Connector_Generic:Conn_02x05_Counter_Clockwise
- added CNA, CNB, CNC: ~, symbol Connector_Generic:Conn_02x16_Counter_Clockwise
- added CN_COIN: Coin discriminator module, symbol Connector_Generic:Conn_02x06_Counter_Clockwise
- added CN_LCD1: LCD module cable connector, symbol Connector_Generic:Conn_02x07_Counter_Clockwise
- added D1, D2 (x2), D3, D4: 1N4148, Diode_THT:D_DO-35_SOD27_P7.62mm_Horizontal, symbol Diode:1N4148
- added D16, D17, D18: ?, Diode_THT:D_DO-41_SOD81_P10.16mm_Horizontal, symbol Diode:1N4007
- added D22, D24, D25: BAS16W, Package_TO_SOT_SMD:SOT-323_SC-70, symbol Diode:BAS16W
- added D23: "225", Package_TO_SOT_SMD:SOT-323_SC-70, symbol Diode:BAS16W
- added H1: ~, symbol IPM_custom:67475
- added H2, H4: ~, symbol IPM_custom:67381
- added H3: 67382, symbol IPM_custom:67382
- added H5: ~, symbol IPM_custom:67384
- added H6, H7, H8: ~, symbol IPM_custom:67383
- added H9: 67476 hybrid, symbol Connector:Conn_01x15_Pin
- added J2: ., symbol Connector:Conn_01x20_Male
- added J3: ~, symbol Connector:Conn_01x15_Pin
- added J4: Conn_02x30_Odd_Even, symbol Connector_Generic:Conn_02x30_Odd_Even
- added JP1: ~, symbol Jumper:Jumper_2_Bridged
- added L1: L_Iron, symbol Device:L_Iron
- added Q10, Q2, Q5, Q7, Q9, Q?: BC847, Package_TO_SOT_SMD:SOT-23, symbol Transistor_BJT:BC847
- added Q11: Si2301, Package_TO_SOT_SMD:SOT-23, symbol Transistor_FET:Si2319CDS
- added Q3, Q4, Q6: BC857, Package_TO_SOT_SMD:SOT-23, symbol Transistor_BJT:BC857
- added Q?: BCW67, Package_TO_SOT_SMD:SOT-23, symbol Transistor_BJT:BC857
- added R1, R3, R5, R?: ~, symbol Device:R
- added R1, R13, R14, R17 (x2), R2, R25, R3, R4, R5, R63, R64, R7, R?: 100k, symbol Device:R
- added R10, R11, R15, R16, R22, R23, R24, R8, R9: ?, symbol Device:R
- added R10, R11, R12, R65, R67, R68: 10k, symbol Device:R
- added R12, R4: 100k?, symbol Device:R
- added R15: 180, symbol Device:R
- added R16, R48, R69: 100, symbol Device:R
- added R18: 100k(?), symbol Device:R
- added R22, R45, R50, R51, R58, R59: 6.5K, symbol Device:R
- added R46, R47: 210, symbol Device:R
- added R49: 10, symbol Device:R
- added R52, R57: 330, symbol Device:R
- added R53, R54, R55, R56: 220, symbol Device:R
- added R6: 47k, symbol Device:R
- added R60: 100K, symbol Device:R
- added R61: 170k, symbol Device:R
- added R62: 11.6k, symbol Device:R
- added R66: 20.8k, symbol Device:R
- added R7: 1.8k, symbol Device:R
- added R8: 22k, symbol Device:R
- added R9: 3.9k, symbol Device:R
- added RN1: AR1, Resistor_THT:R_Array_SIP9, symbol Device:R_Network08
- added SUR1: ~, symbol IPM_custom:LIOD_PSU
- added SW12: SW_SPST, symbol Switch:SW_SPST
- added T1, T2, T3, T4, T5: BC337, Package_TO_SOT_THT:TO-92_Inline, symbol Transistor_BJT:BC337
- added U10: 4023, symbol 4xxx:4023
- added U11, U4: 4001, symbol 4xxx:4001
- added U12: ITR9608-F, OptoDevice:Everlight_ITR9608-F, symbol Sensor_Proximity:ITR9608-F
- added U2, U9: 74LS125, symbol 74xx:74LS125
- added U3, U4: 74HC244, symbol 74xx:74HC244
- added U5: HEF4093B, symbol 4xxx:HEF4093B
- added U6: 74HC373, symbol 74xx:74HC373
- added U6: 74HC14, symbol 74xx:74HC14
- added U7: 74LS148, symbol 74xx:74LS148
- added U8: 4556, symbol 4xxx_IEEE:4556
- D1: value "1FK" -> 1FK; Spice_Netlist_Enabled Y -> (none); Spice_Primitive D -> (none)
- D3: value 1N4007 -> ?
- renumbered CN1 to CN1L, CN1 to CN1_L, CN2 to CN2_L, CN3 to CN3_L, CN5 to CN5_L, CN6 to CN6_L
Connections:
- net CN3-5 is gone; now on net +BATT: CN1L.7 (Pin_7)
- net +5V: now also R?.1, U1.20 (VCC), U2.14 (VCC), AR2.1 (common), C10.2, C11.2, C12.2, C13.1, C6.2, C7.2, C8.2, C9.2, CN1.2 (Pin_2), CN1.43 (Pin_43), CN1.47 (Pin_47), CN1.9 (Pin_9), CN2.12 (Pin_12), CN2.29 (Pin_29), CN3L1.8 (Pin_8), CNA.16 (Pin_16), CNA.17 (Pin_17), CNA.3 (Pin_3), CNA.30 (Pin_30), CNC.23 (Pin_23), H2.4 (VCC), H3.9 (VCC), H4.4 (VCC), H5.4 (VCC), H6.8 (VCC), H7.8 (VCC), H8.8 (VCC), H9.7 (Pin_7), J2.4 (Pin_4), J3.7 (Pin_7), R1.1, R1.1, R10.1, R11.1, R11.1, R12.1, R13.1, R14.1, R2.1, R25.1, R3.1, R4.1, R5.1, R63.1, R64.1, R7.1, R8.1, R?.1, RN1.1 (common), U10.14 (VDD), U10.2, U10.8, U11.14 (VDD), U3.20 (VCC), U4.14 (VDD), U4.20 (VCC), U5.14 (VCC), U5.20 (VCC), U6.14 (VCC), U6.20 (VCC), U7.16 (VCC), U8.16 (Vdd), U8.8 (Vss), U9.14 (VCC)
- net +BATT: now also C14.1, CN1.36 (Pin_36), CN1.42 (Pin_42), CN1.44 (Pin_44), CN1.46 (Pin_46), CN2.13 (Pin_13), CN2.28 (Pin_28), CN3L1.5 (Pin_5), H1.13 (VBAT), H5.15 (VBAT1), H5.16 (VBAT2), J2.15 (Pin_15), J2.16 (Pin_16), Q3.2 (E), R16.1, R46.1, SUR1.1 (VBAT); no longer Q8.2 (E)
- net GND: now also J?.12 (Pin_12), U1.10 (GND), U2.7 (GND), C1.1, C10.1, C11.1, C12.1, C13.2, C14.2, C2.1, C2.1, C22.1, C3.1, C4.1, C5.1, C6.1, C7.1, C8.1, C9.1, CN1.16 (Pin_16), CN1.20 (Pin_20), CN1.22 (Pin_22), CN1.26 (Pin_26), CN1.29 (Pin_29), CN1.52 (Pin_52), CN1.59 (Pin_59), CN1.60 (Pin_60), CN2.11 (Pin_11), CN2.30 (Pin_30), CN2L.4 (Pin_4), CN2L.7 (Pin_7), CN3L1.4 (Pin_4), CN3L1.7 (Pin_7), CNA.1 (Pin_1), CNA.32 (Pin_32), CNC.1 (Pin_1), CNC.16 (Pin_16), CNC.17 (Pin_17), CNC.32 (Pin_32), D16.2 (A), D18.2 (A), D23.1 (A), D24.1 (A), H1.14 (GND), H2.12 (GND), H3.5 (GND), H4.12 (GND), H5.1 (GND1), H5.10 (GND6), H5.17 (GND7), H5.2 (GND2), H5.20 (GND8), H5.6 (GND3), H5.8 (GND4), H5.9 (GND5), H6.10 (GND2), H6.5 (GND1), H7.10 (GND2), H7.5 (GND1), H8.10 (GND2), H8.5 (GND1), H9.1 (Pin_1), H9.14 (Pin_14), J2.1 (Pin_1), J2.10 (Pin_10), J2.11 (Pin_11), J2.17 (Pin_17), J2.2 (Pin_2), J2.20 (Pin_20), J2.6 (Pin_6), J2.8 (Pin_8), J2.9 (Pin_9), J3.1 (Pin_1), J3.14 (Pin_14), Q11.3 (D), Q2.2 (E), Q4.3 (C), Q7.2 (E), Q9.2 (E), R12.2, R15.2, R17.2, R17.2, R18.2, R23.2, R4.2, R45.2, R5.1, R51.2, R53.1, R56.1, R58.2, R60.1, R62.1, R65.2, R67.2, R68.1, R7.1, R9.2, SUR1.2 (GND1), SUR1.4 (GND2), T1.3 (E), T2.3 (E), T3.3 (E), T4.3 (E), T5.3 (E), U10.7 (VSS), U11.7 (VSS), U3.10 (GND), U4.10 (GND), U4.7 (VSS), U5.10 (GND), U5.7 (GND), U6.10 (GND), U6.7 (GND), U7.10 (IO), U7.4 (I7), U7.8 (GND), U8.16 (Vdd), U8.8 (Vss), U9.7 (GND)
- net KBD_1: now also CN2.2 (Pin_2), D1.2 (A)
- net KBD_2: now also CN2.1 (Pin_1), D4.2 (A)
- net KBD_3: now also CN2.40 (Pin_40), CNB.15 (Pin_15), R10.2
- net KBD_4: now also CN2.39 (Pin_39), D3.2 (A); no longer SW1.1, SW4.1, SW7.1, SW9.1
- net KBD_5: now also SW1.1, SW4.1, SW7.1, SW9.1, CN2.3 (Pin_3), CNB.16 (Pin_16), R12.2; no longer SW1.2, SW2.2, SW3.2
- net KBD_6: now also SW1.2, SW2.2, SW3.2, CN2.38 (Pin_38), D2.2 (A); no longer SW10.1, SW2.1, SW5.1, SW8.1
- net KBD_7: now also SW10.1, SW2.1, SW5.1, SW8.1, CN2.4 (Pin_4), CNB.18 (Pin_18), R11.2
- net ~{RST}: now also CN1.1 (Pin_1), CNA.2 (Pin_2)
- net at D3.1 (K): now also Q8.2 (E), D17.1 (K), Q3.3 (C), Q4.2 (E), Q6.2 (E), R48.1, R54.2, R55.2
- net at D3.2 (A): now also D16.1 (K), J2.12 (Pin_12), Q6.3 (C), Q7.3 (C); no longer Q8.3 (C)
- net CN1L-5: now reaches CN1L.5 (Pin_5)
- net CN1L-5: now also CN2L.2 (Pin_2), CN3L1.2 (Pin_2), R22.1, R23.1, T1.2 (B)
- net at CN1L.6 (Pin_6): now also SUR1.3 (UNK)
- net at U2.12: now also U1.8 (1A3), U3.15 (Reset)
- net at J?.12 (Pin_12), R?.1: now also Q?.2 (E)
- net at R?.1, R?.2: now also Q?.1 (B)
- net at SWR.3 (C): now also CN2B.11 (Pin_11); no longer CN2B.10 (Pin_10)
- net at U2.8: now also U1.19 (2OE)
- net at U2.9: now also U1.1 (1OE), U2.10
- net at J1.1 (Pin_1), U1.1, U1.12: now also R60.2; no longer C?.1
- net at J1.7 (Pin_7), U1.13: now also C?.1, R?.2
- net at Q1.1 (B): now also R22.2, R45.1
- net at U2.1: now also U3.14 (CLK), R1.2, T2.1 (C)
- net at U2.2: now also R6.2
- net at SWH.5 (B): now also CN2B.10 (Pin_10); no longer CN2B.9 (Pin_9)
- net at Q8.1 (B): now also R52.1, R55.1
- net at J?.13 (Pin_13): now also Q?.3 (C)
- net SAFE_SW2: now reaches C16.2, CN1_L.20 (Pin_20)
- net SAFE_SW2: now also R32.2, AR2.7 (R6), CN2.20 (Pin_20), U3.15 (2A1); no longer R32.1
- net at R?.2: now also Q?.3 (C)
- net at CN6.2 (Pin_2), CN6.4 (Pin_4): now also R32.1; no longer R32.2
- net at U2.5: now also U2.4
- net at U2.6: now also U2.11, C1.1
- net at U1.11 (2A3): now also U1.5 (2Y1), R7.2
- net LIOD_RESET: now reaches U1.12 (1Y3)
- net LIOD_RESET: now also CN3L1.10 (Pin_10)
- net at U1.13 (2A2): now also R11.2, T4.1 (C)
- net at U1.14 (1Y2): now also U1.2 (1A0), R5.2
- net at U1.15 (2A1): now also R?.2, T5.1 (C)
- net ~{LIOD_RESET_BUFF}: now reaches U1.3 (2Y0)
- net ~{LIOD_RESET_BUFF}: now also R25.2, R8.1
- net at U1.4 (1A1): now also CN3L1.3 (Pin_3), R18.1
- net at U1.6 (1A2): now also CN3L1.1 (Pin_1), R17.1
- net at J?.14 (Pin_14), R?.1: now also Q?.2 (E)
- net at J1.9 (Pin_9), Q?.3 (C): no longer R?.2
- net at J1.2 (Pin_2), R?.2, U1.2: now also C?.1
- net at Q1.3 (C): now also R47.2
- net at R?.2, R?.2: now also Q?.1 (B)
- net SAFE_SW1: now reaches C17.2, CN1_L.19 (Pin_19), R33.1
- net SAFE_SW1: now also AR2.3 (R2), CN2.19 (Pin_19), U4.11 (2A3)
- net at U2.3: now also C1.2, R6.1
- net at D1.2 (A), R21.2: now also CN2L.9 (Pin_9)
- net at U3.9 (Q8): now also R22.2
- net CN1-1 renamed CN1L-1
- net CN1-2 renamed ~{LIOD_RESET}
- net CN1-26 renamed ~{I_LIMIT}
- net ~{I_LIMIT}: now also CN2.26 (Pin_26), CNA.12 (Pin_12), R1.2
- net CN1-3 renamed CN1L-3
- net CN1-31 renamed AC_DIN
- net AC_DIN: now also CN2.31 (Pin_31)
- net CN1-33 renamed AS_DIN
- net AS_DIN: now also CN2.33 (Pin_33), JP1.1 (A)
- net CN1-35 renamed RL2-S
- net RL2-S: now also CN2.35 (Pin_35), H1.10 (OUT)
- net CN1-37 renamed RL1-S
- net RL1-S: now also CN2.37 (Pin_37), H2.11 (OUT)
- net CN1-4 renamed CN1L-4
- net CN1L-4: now also D2.1 (K)
- net CN1-6 renamed RL1-R
- net RL1-R: now also CN2.6 (Pin_6), H2.13 (OUT)
- net CN1-7 renamed RL2-R
- net RL2-R: now also CN2.7 (Pin_7), H1.7 (OUT)
- net CN1-8 renamed AS_DOUT
- net AS_DOUT: now also CN2.8 (Pin_8), H1.3 (OUT)
- net CN1-9 renamed AC_DOUT
- net AC_DOUT: now also CN2.9 (Pin_9), H1.1 (OUT)
- net CN2-1 renamed CN2L-1
- net CN2L-1: now also CN2L.1 (Pin_1), R3.2, R?.2
- new net: H9.4 (Pin_4), JP1.2 (B), R5.2
- new net: CN2L.8 (Pin_8), R10.1
- new net: CN2L.10 (Pin_10), R10.2, T3.1 (C)
- new net: Q3.1 (B), R46.2, R47.1
- new net: H4.6 (OUT), H6.1 (IN1)
- new net: H6.4 (IN2), U6.15 (O5)
- new net: H4.10 (IN), U2.1, U2.10, U2.13, U2.4, U8.5 (~{Q1})
- new net: H3.2 (OUT), U2.5
- new net: C21.1, D24.3 (K), R67.1, U6.1
- new net: R3.1, R4.1, T2.2 (B)
- new net: Q6.1 (B), R54.1, R57.1
- new net: CN_LCD1.1 (Pin_1), J4.1 (Pin_1)
- new net: CN_LCD1.10 (Pin_10), J4.10 (Pin_10)
- new net: CN_LCD1.11 (Pin_11), J4.8 (Pin_8)
- new net: CN_LCD1.12 (Pin_12), J4.6 (Pin_6)
- new net: CN_LCD1.13 (Pin_13), J4.4 (Pin_4)
- new net: CN_LCD1.14 (Pin_14), J4.2 (Pin_2)
- new net: CN_LCD1.2 (Pin_2), J4.3 (Pin_3)
- new net: CN_LCD1.3 (Pin_3), J4.5 (Pin_5)
- new net: CN_LCD1.4 (Pin_4), J4.7 (Pin_7)
- new net: CN_LCD1.5 (Pin_5), J4.9 (Pin_9)
- new net: CN_LCD1.6 (Pin_6), J4.11 (Pin_11)
- new net: CN_LCD1.7 (Pin_7), J4.13 (Pin_13)
- new net: CN_LCD1.8 (Pin_8), J4.14 (Pin_14)
- new net: CN_LCD1.9 (Pin_9), J4.12 (Pin_12)
- new net: H7.4 (IN2), U6.9 (O3)
- new net: R15.1, R16.1, T5.2 (B)
- new net: CN2L.5 (Pin_5), SUR1.5 (UNK2)
- new net: H1.15 (IN), H9.3 (Pin_3)
- new net: D23.3 (K), R61.2, R66.2, U5.5
- new net: H4.9 (IN), U4.1 (1OE), U4.19 (2OE), U8.7 (~{Q3})
- new net: H2.7 (OUT1), U4.13 (2A2)
- new net: H3.6 (OUT), U4.15 (2A1)
- new net: H2.6 (OUT), U4.17 (2A0)
- new net: U4.2 (1A0), U7.9 (S0)
- new net: U4.4 (1A1), U7.7 (S1)
- new net: U4.6 (1A2), U7.6 (S2)
- new net: R50.1, U4.4
- new net: Q5.1 (B), R50.2, R51.1
- new net: C2.2, CN3L1.9 (Pin_9), D2.2 (A), R24.1
- new net: H5.7 (DRV_EN), U11.4
- new net: C5.2, Q11.1 (G), R62.2, U5.8, U5.9
- new net: D4.1 (K), U8.10 (~{Q2})
- new net: D1.1 (K), U8.11 (~{Q1})
- new net: D2.1 (K), U8.12 (~{Q0})
- new net: D3.1 (K), U8.9 (~{Q3})
- new net: C21.2, U6.3, U6.6
- new net: U11.10, U11.5
- new net: J3.10 (Pin_10), U6.8
- new net: J3.11 (Pin_11), U6.4
- new net: J3.12 (Pin_12), U6.2
- new net: J3.13 (Pin_13), R69.1
- new net: J3.2 (Pin_2), U5.6
- new net: J3.3 (Pin_3), R61.1, U5.3
- new net: J3.4 (Pin_4), R63.2, U5.12
- new net: J3.5 (Pin_5), U5.10
- new net: J3.6 (Pin_6), R64.2, U5.13
- new net: J3.8 (Pin_8), U6.13
- new net: J3.9 (Pin_9), U6.10
- new net: H3.10 (IN), R7.2, R9.2
- new net: C19.1, U6.11, U6.12
- new net: D22.3 (K), U5.1, U5.2, U5.4
- new net: J2.7 (Pin_7), U4.1, U4.2
- new net: U4.13, U4.3, U4.5, U4.9
- new net: J2.3 (Pin_3), Q2.1 (B), U4.12
- new net: Q2.3 (C), R49.2
- new net: Q4.1 (B), R48.2, R49.1
- new net: D25.1 (A), R69.2
- new net: C22.2, D25.3 (K), R68.2, U6.5
- new net: Q10.3 (C), R57.2
- new net: C5.1, U5.11
- new net: D17.2 (A), D18.1 (K), J2.18 (Pin_18), Q8.3 (C), Q9.3 (C)
- new net: C19.2, Q11.2 (S), R65.1, U6.9
- new net: H9.12 (Pin_12), U10.3
- new net: H9.10 (Pin_10), U10.4
- new net: H9.5 (Pin_5), U10.5
- new net: U10.12, U10.6
- new net: Q5.2 (E), Q7.1 (B), R53.2
- new net: CN1.40 (Pin_40), R16.2
- new net: Q5.3 (C), R52.2
- new net: R12.1, R?.1, T4.2 (B)
- new net: Q10.2 (E), Q9.1 (B), R56.2
- new net: R22.1, U4.11
- new net: R8.2, R9.1, T3.2 (B)
- new net: H3.7 (OUT), U2.9
- new net: U3.1 (1OE), U3.19 (2OE), U8.6 (~{Q2})
- new net: H4.7 (OUT1), U3.13 (2A2)
- new net: Q10.1 (B), R58.1, R59.1
- new net: R59.2, U4.10, U4.6
- new net: J2.5 (Pin_5), U4.8
- new net: H3.4 (OUT), U2.12
- new net: R24.2, T1.1 (C)
- new net: D22.1 (A), R66.1
- new net B_A0: CNB.21 (Pin_21), U5.3 (D0), U6.3 (D0)
- new net B_A1: CNB.12 (Pin_12), U5.4 (D1), U6.4 (D1)
- new net B_A2: CNB.22 (Pin_22), U5.7 (D2), U6.7 (D2)
- new net B_A3: CNB.11 (Pin_11), U5.8 (D3), U6.8 (D3)
- new net B_A4: CNB.23 (Pin_23), U5.13 (D4), U6.13 (D4)
- new net B_A5: CNB.10 (Pin_10), U5.14 (D5), U6.14 (D5)
- new net B_A6: CNB.24 (Pin_24), U5.17 (D6), U6.17 (D6)
- new net B_A7: CNB.9 (Pin_9), U5.18 (D7), U6.18 (D7)
- new net CN1-21: CN1.21 (Pin_21), CN1.38 (Pin_38)
- new net CN1-23: CN1.23 (Pin_23), CN1.31 (Pin_31)
- new net CN1-53: CN1.53 (Pin_53), H9.8 (Pin_8)
- new net CN2-16: H9.6 (Pin_6)
- new net CN2-18: CN2.18 (Pin_18), CNC.14 (Pin_14)
- new net CN2-21: U11.12, U11.3
- new net CN2-22: CN2.22 (Pin_22), H4.11 (OUT), R15.2
- new net CN2-31: R17.1, U10.1
- new net CN2-34: CN2.34 (Pin_34), H1.5 (OUT)
- new net CN2L-3: CN2L.3 (Pin_3), R16.2
- new net COIN_D0: CN1.51 (Pin_51), U7.5 (EI)
- new net COIN_D1: CN1.48 (Pin_48), U7.11 (I1)
- new net COIN_D2: CN1.11 (Pin_11), U7.12 (I2)
- new net COIN_D3: CN1.50 (Pin_50), U7.13 (I3)
- new net COIN_D4: CN1.12 (Pin_12), U7.1 (I4)
- new net COIN_D5: CN1.49 (Pin_49), U7.2 (I5)
- new net COIN_D6: CN1.13 (Pin_13), U7.3 (I6)
- new net COIN_SW1: CN2.10 (Pin_10), H2.3 (IN)
- new net COIN_SW2: CN2.32 (Pin_32), H2.2 (IN)
- new net C_A0: CNC.28 (Pin_28), U5.2 (O0)
- new net C_A1: CNC.7 (Pin_7), U5.5 (O1)
- new net C_A10: CNC.27 (Pin_27)
- new net C_A2: CNC.26 (Pin_26), U5.6 (O2)
- new net C_A3: CNC.8 (Pin_8), U5.9 (O3)
- new net C_A4: CNC.25 (Pin_25), U5.12 (O4)
- new net C_A5: CNC.24 (Pin_24), U5.15 (O5)
- new net C_A6: CNC.10 (Pin_10), U5.16 (O6)
- new net C_A7: CNC.22 (Pin_22), U5.19 (O7)
- new net C_A8: CNC.11 (Pin_11), U6.2 (O0)
- new net C_A9: CNC.9 (Pin_9), U6.12 (O4)
- new net C_D0: CNB.1 (Pin_1), CNC.29 (Pin_29), RN1.3 (R2), U3.18 (1Y0), U4.18 (1Y0)
- new net C_D1: CNB.32 (Pin_32), CNC.31 (Pin_31), RN1.5 (R4), U3.16 (1Y1), U4.16 (1Y1)
- new net C_D2: CNB.2 (Pin_2), CNC.2 (Pin_2), RN1.7 (R6), U3.14 (1Y2), U4.14 (1Y2)
- new net C_D3: CNB.31 (Pin_31), CNC.3 (Pin_3), RN1.9 (R8), U3.12 (1Y3), U4.12 (1Y3)
- new net C_D4: CNB.3 (Pin_3), CNC.30 (Pin_30), RN1.8 (R7), U2.3, U3.9 (2Y3), U4.9 (2Y3)
- new net C_D5: CNB.30 (Pin_30), CNC.4 (Pin_4), H2.5 (OUT), RN1.6 (R5), U2.6, U3.7 (2Y2), U4.7 (2Y2)
- new net C_D6: CNB.4 (Pin_4), CNC.5 (Pin_5), RN1.4 (R3), U2.8, U3.5 (2Y1), U4.5 (2Y1)
- new net C_D7: CNB.29 (Pin_29), CNC.6 (Pin_6), RN1.2 (R1), U2.11, U3.3 (2Y0), U4.3 (2Y0)
- new net C_S0: CNC.19 (Pin_19), U6.5 (O1)
- new net C_S1: CNC.21 (Pin_21), U6.6 (O2)
- new net C_S2: CNC.15 (Pin_15)
- new net ENC0: AR2.5 (R4), C1.2, CN1.35 (Pin_35), U3.2 (1A0)
- new net ENC1: AR2.4 (R3), C2.2, CN1.27 (Pin_27), U3.4 (1A1)
- new net ENC2: AR2.6 (R5), C3.2, CN1.34 (Pin_34), U3.6 (1A2)
- new net ENC3: AR2.8 (R7), C4.2, CN1.28 (Pin_28), U3.8 (1A3)
- new net ENC4: AR2.9 (R8), C5.2, CN1.33 (Pin_33), U3.11 (2A3)
- new net FS_LED: CN1.6 (Pin_6), H1.13 (OUT)
- new net H4-3: H4.3 (IN), H4.5 (OUT), U3.17 (2A0)
- new net H4-8: H4.8 (OUT2), H7.1 (IN1)
- new net H8-4: H8.4 (IN2), U6.16 (O6)
- new net H9-11: H9.11 (Pin_11), U4.8 (1A3)
- new net H9-15: CN2.36 (Pin_36), H9.15 (Pin_15)
- new net H9-2: H9.2 (Pin_2), U11.11
- new net HOOK: AR2.2 (R1), CN2.17 (Pin_17), U2.2
- new net LCD_CLK: CN1.3 (Pin_3), CNA.10 (Pin_10)
- new net LCD_C/~{D}: CN1.5 (Pin_5), CNA.8 (Pin_8)
- new net LCD_MOSI: CN1.57 (Pin_57), CNA.24 (Pin_24)
- new net MCU-PC0: U5.1 (OE), U6.1 (OE)
- new net PA0: CNA.26 (Pin_26), H1.2 (IN)
- new net PA1: CNA.7 (Pin_7), H1.8 (IN)
- new net PA2: CNA.27 (Pin_27), H1.11 (IN)
- new net PA3: CNA.6 (Pin_6), U10.9
- new net PA4: CNA.28 (Pin_28), H1.4 (IN)
- new net PA5: CNA.5 (Pin_5)
- new net PA6: CNA.29 (Pin_29), U8.14 (A0)
- new net PA7: CNA.4 (Pin_4), U8.13 (A1)
- new net PB0: CNA.22 (Pin_22), U11.1, U11.2
- new net PB1: CNA.11 (Pin_11), H1.6 (IN)
- new net PB2: CNA.23 (Pin_23), H2.9 (IN)
- new net PC0: CN2.23 (Pin_23), CNA.18 (Pin_18), U10.11, U10.13, U11.13, U11.6, U8.1 (~{EN}), U8.15 (~{EN})
- new net PC1: CN1.10 (Pin_10), CNA.15 (Pin_15)
- new net PC2: CNA.19 (Pin_19), CNC.18 (Pin_18), R2.2
- new net PC3: CNA.14 (Pin_14), H8.1 (IN1)
- new net PC4: CNA.20 (Pin_20), H2.10 (IN)
- new net PC5: CN2.25 (Pin_25), CNA.13 (Pin_13), R3.2
- new net PC6: CN2.27 (Pin_27), CNA.21 (Pin_21), R4.2
- new net PD4: CNB.19 (Pin_19), H9.9 (Pin_9)
- new net PD5: CNB.14 (Pin_14)
- new net PHOTO_POCKET: CN1.39 (Pin_39), H3.8 (IN)
- new net PHOTO_R_EXIT: CN1.45 (Pin_45), R8.2, R9.1
- new net PHOTO_R_IN: CN1.32 (Pin_32), H3.1 (IN)
- new net PHOTO_R_IN_PWR: CN1.30 (Pin_30), CN2.24 (Pin_24), H4.13 (OUT)
- new net PHOTO_R_POCKET_PWR: CN1.17 (Pin_17), R15.1
- new net PHOTO_SAFE: CN1.41 (Pin_41), H3.3 (IN)
- new net REDIAL: CN2.5 (Pin_5), H2.1 (IN)
- new net R_MOT_A: CN1.24 (Pin_24), H5.18 (MOT2)
- new net R_MOT_B: CN1.37 (Pin_37), H5.12 (MOT1)
- new net SCL-39: CN2.15 (Pin_15), CNB.17 (Pin_17)
- new net SCL-43: CNB.25 (Pin_25), U11.8, U11.9
- new net SCL-44: CNB.8 (Pin_8), H5.5 (DIR)
- new net SCL-45: CNB.26 (Pin_26), H5.3 (~{RUN}/STOP)
- new net SCL-46: CN2.14 (Pin_14), CNB.7 (Pin_7)
- new net SCL-47: CNB.27 (Pin_27), U5.11 (LE)
- new net SCL-50: CNB.6 (Pin_6), U6.11 (LE)
- new net SCL-51: CNB.28 (Pin_28), U8.2 (A0)
- new net SCL-52: CNB.5 (Pin_5), U8.3 (A1), U8.4 (~{Q0})
- new net SOLENOID_C_PATH: CN1.19 (Pin_19), H6.9 (SOL)
- new net SOLENOID_C_REJ: CN1.15 (Pin_15), H7.9 (SOL)
- new net SOLENOID_R_POCKET: CN1.25 (Pin_25), H8.9 (SOL)
- new net SW1: CN1.54 (Pin_54), CNB.13 (Pin_13), R14.2
- new net SW2: CN1.7 (Pin_7), CNB.20 (Pin_20), R13.2
- new net SW_C_PATH: CN1.18 (Pin_18), H4.1 (IN)
- new net SW_C_REJ: CN1.14 (Pin_14), H4.2 (IN)
- new net ~{IRQ}: CNA.31 (Pin_31), U10.10
- new net ~{LCD_BUSY}: CN1.56 (Pin_56), CNA.25 (Pin_25)
- new net ~{LCD_CS}: CN1.4 (Pin_4), CNA.9 (Pin_9)
- new net ~{LCD_RESET}: CN1.55 (Pin_55), U6.19 (O7)
- no-connect marks 0 -> 37
Other:
- added sheet 67476 (modules_67476.kicad_sch)
- added sheet Main board (rotor_main.kicad_sch)
- note added: "Coin disc."
- note added: "Coin path solenoid"
- note added: "Coin path switch"
- note added: "Coin reject solenoid"
- note added: "Coin reject sw"
- note added: "Coin-in-safe photointerrupter"
- note added: "Hookswitch"
- note added: "LCD"
- note added: "No designators present on module. Resistors are thick-film on ceramic, laser trimmed. Reported values are direct measures."
- note added: "Power"
- note added: "Rotor absolute encoder"
- note added: "Rotor exit photointerrupter"
- note added: "Rotor input photointerrupter"
- note added: "Rotor motor"
- note added: "Rotor pocket photointerrupter"
- note added: "Rotor pocket solenoid"
- moved on the sheet: C11, C16, C17, C?, CN1L, CN2B, CN6, CN_LCD, CN_LCD2, D1, DL1, J1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

Commit message: Fixed some errors on the main board schematic
Parts:
- removed CN_LCD1: LCD module cable connector, symbol Connector_Generic:Conn_02x07_Counter_Clockwise
- removed J4: Conn_02x30_Odd_Even, symbol Connector_Generic:Conn_02x30_Odd_Even
- removed SW12: SW_SPST, symbol Switch:SW_SPST
- added CN_LCD: LCD module cable connector, symbol Connector_Generic:Conn_02x07_Counter_Clockwise
- added M1: Rotor motor, symbol Motor:Motor_DC
- added OPT2: Coin tray entrance photointerrupter, OptoDevice:Everlight_ITR9608-F, symbol Sensor_Proximity:ITR9608-F
- added OPT3: "Rotor pocket open" photointerrupter, OptoDevice:Everlight_ITR9608-F, symbol Sensor_Proximity:ITR9608-F
- added OPT4: Rotor pocket entrance photointerrupter, OptoDevice:Everlight_ITR9608-F, symbol Sensor_Proximity:ITR9608-F
- added R16: 100, symbol Device:R
- added SOL2: Coin path solenoid, symbol Device:L_Iron
- added SOL3: Coin rotor pocket open/close solenoid, symbol Device:L_Iron
- added SW_C_PATH: Coin path switch, symbol Switch:SW_SPST
- added SW_ENC0, SW_ENC1, SW_ENC2, SW_ENC3, SW_ENC4: Rotor absolute position encoder, symbol Switch:SW_SPST
- added SW_REJ: Coin reject actuator switch, symbol Switch:SW_SPST
- OPT1: renamed from U12; value ITR9608-F -> Rotor pocket exit photointerrupter
- SOL1: renamed from L1; value L_Iron -> Coin reject solenoid
Connections:
- net +5V: now also CN_COIN.1 (Pin_1), CN_LCD.2 (Pin_2), SW_C_PATH.2 (B), SW_REJ.2 (B)
- net +BATT: now also OPT1.1, SOL1.2, R16.1, SOL2.2, SOL3.2
- net CN1-21: now also OPT2.2, OPT3.1
- net CN1-23: now also OPT3.2, OPT4.1
- net CN1-53: now also CN_COIN.6 (Pin_6)
- net CN1L-5: no longer R22.1, R23.1, T1.2 (B)
- net COIN_D0: now also CN_COIN.5 (Pin_5)
- net COIN_D1: now also CN_COIN.2 (Pin_2)
- net COIN_D2: now also CN_COIN.9 (Pin_9)
- net COIN_D3: now also CN_COIN.4 (Pin_4)
- net COIN_D4: now also CN_COIN.10 (Pin_10)
- net COIN_D5: now also CN_COIN.3 (Pin_3)
- net COIN_D6: now also CN_COIN.11 (Pin_11)
- net ENC0: now also SW_ENC0.1 (A)
- net ENC1: now also SW_ENC1.1 (A)
- net ENC2: now also SW_ENC2.1 (A)
- net ENC3: now also SW_ENC3.1 (A)
- net ENC4: now also SW_ENC4.1 (A)
- net FS_LED: now also CN_LCD.6 (Pin_6)
- net GND: now also OPT1.4, CN_LCD.13 (Pin_13), CN_LCD.14 (Pin_14), OPT2.4, OPT3.4, OPT4.4, SW_ENC0.2 (B), SW_ENC1.2 (B), SW_ENC2.2 (B), SW_ENC3.2 (B), SW_ENC4.2 (B)
- net LCD_CLK: now also CN_LCD.3 (Pin_3)
- net LCD_C/~{D}: now also CN_LCD.5 (Pin_5)
- net LCD_MOSI: now also CN_LCD.11 (Pin_11)
- net PC1: now also CN_COIN.8 (Pin_8)
- net PHOTO_POCKET: now also OPT3.3
- net PHOTO_R_EXIT: now also OPT1.3
- net PHOTO_R_IN: now also OPT4.3
- net PHOTO_R_IN_PWR: now also OPT4.2
- net PHOTO_R_POCKET_PWR: now also OPT1.2
- net PHOTO_SAFE: now also OPT2.3
- net R_MOT_A: now also M1.1 (+)
- net R_MOT_B: now also M1.2 (-)
- net SOLENOID_C_PATH: now also SOL2.1
- net SOLENOID_C_REJ: now also SOL1.1
- net SOLENOID_R_POCKET: now also SOL3.1
- net SW1: now also CN_LCD.8 (Pin_8)
- net SW2: now also CN_LCD.7 (Pin_7)
- net SW_C_PATH: now also SW_C_PATH.1 (A)
- net SW_C_REJ: now also CN_COIN.12 (Pin_12), SW_REJ.1 (A)
- net ~{LCD_BUSY}: now also CN_LCD.10 (Pin_10)
- net ~{LCD_CS}: now also CN_LCD.4 (Pin_4)
- net ~{LCD_RESET}: now also CN_LCD.9 (Pin_9)
- net ~{RST}: now also CN_LCD.1 (Pin_1)
- new net: R22.1, R23.1, T1.2 (B)
- new net: OPT2.1, R16.2
- no-connect marks 37 -> 39
Other:
- note added: "This solenoid opens the currently selected coin rotor pocket to dump out its contents."
- note added: "This solenoid selects whether the coin coming out from the coin rotor's pocket is directed to the coin box or to the coin return tray"
- note added: "This solenoid selects whether the coin is directed to the coin rotor (if accepted) or to the coin return tray (if rejected)"
- note removed: "Coin disc."
- note removed: "Coin path solenoid"
- note removed: "Coin path switch"
- note removed: "Coin reject solenoid"
- note removed: "Coin reject sw"
- note removed: "Coin-in-safe photointerrupter"
- note removed: "LCD"
- note removed: "Rotor absolute encoder"
- note removed: "Rotor exit photointerrupter"
- note removed: "Rotor input photointerrupter"
- note removed: "Rotor motor"
- note removed: "Rotor pocket photointerrupter"
- note removed: "Rotor pocket solenoid"
- moved on the sheet: OPT1, SOL1

Commit message: Fixed minor mistakes in the schematics
Parts:
- ML1: symbol IPM_custom:64357/A -> IPM_custom:64357/A
- renumbered U11 to U1, U9 to U2, U10 to U9
Connections:
- net CN2-31 is gone; now on net AC_DIN: R17.1, U9.1
- net CN2-16: now also CN2.16 (Pin_16)
- net at J3.13 (Pin_13): no longer R69.1
- net at J3.15 (Pin_15): now also R69.1
- no-connect marks 39 -> 42

Commit message: Fixed mistakes in main board schematics
Parts:
- added R6: ~, symbol Device:R
Connections:
- net PA5 is gone; now on net AS_DIN: CNA.5 (Pin_5)
- net +5V: now also R6.1
- net AS_DIN: now also R6.2
- net CN1L-5: now also R22.1, R23.1, T1.2 (B)
Other:
- moved on the sheet: AR2, C1, C10, C11, C12, C13, C14, C15, C16, C17, C18, C19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

Commit message: Schematics update
Connections:
- net CN1L-5: no longer R22.1, R23.1, T1.2 (B)
- net COUNTER_RST: now reaches CN1_L.10 (Pin_10), CN5_L.4 (Pin_4)
- net TRAY_FULL: now reaches CN1_L.32 (Pin_32), CN5_L.2 (Pin_2)
- net LIOD_RESET renamed ~{CN1L-2}
- net ~{LIOD_RESET_BUFF} renamed CN1L-2_BUFF
- net ~{LIOD_RESET} renamed CN1L-2
- new net: R22.1, R23.1, T1.2 (B)
Other:
- moved on the sheet: CN5_L, R22

Commit message: Updated schematics
Parts:
- gave numbers to parts that had none: 1
Connections:
- net MCU-PC0 is gone; now on net PC0: U5.1 (OE), U6.1 (OE)
- net SCL-52: no longer U8.4 (~{Q0})
- net DET: now reaches CN3L1.3 (Pin_3), R18.1, U1.4 (1A1)
- net ~{TXD}: now reaches CN3L1.1 (Pin_1), R17.1, U1.6 (1A2)
- net C_S0 renamed ~{EXT_WR}
- net C_S1 renamed ~{EXT_ROM}
- net C_S2 renamed ~{EXT_SEL}
- net ~{EXT_SEL}: now also U8.4 (~{Q0})
- net H8-4: no longer names the net of H8.4 (IN2), U6.16 (O6)
- net SCL-39 renamed SCL-49
Other:
- moved on the sheet: U8A

Commit message: Updated the Line Interface card schematic: fixed mistakes on front panel connections, added some info about the external safe connector
Parts:
- added OPT5: Coin return tray sensor (optional), OptoDevice:Everlight_ITR9608-F, symbol Sensor_Proximity:ITR9608-F
Connections:
- net CN2-22: no longer CN2.22 (Pin_22)
- net H9-15: no longer H9.15 (Pin_15)
- net HOOK: now also CN1_L.36 (Pin_36), CN2_L.9 (Pin_9); no longer CN2.17 (Pin_17), U2.2
- net REDIAL: now also CN1_L.5 (Pin_5), CN2_L.11 (Pin_11)
- net PHOTO_RET_TRAY: now reaches CN1_L.17 (Pin_17), T11.1 (C)
- net PHOTO_RET_TRAY: now also CN2.17 (Pin_17), U2.2
- net at SWR.2 (B): now also CN2B.6 (Pin_6); no longer CN2B.7 (Pin_7)
- net at SWH.5 (B): now also CN2B.9 (Pin_9); no longer CN2B.10 (Pin_10)
- net PHOTO_RET_TRAY_PWR: now reaches CN2_L.7 (Pin_7), R39.2
- net SAFE_TRAY_SW: now reaches CN1_L.22 (Pin_22), CN6.5 (Pin_5)
- net SAFE_TRAY_SW: now also CN2.22 (Pin_22), H9.15 (Pin_15)
- net RET_TRAY: now reaches CN2_L.10 (Pin_10), R40.1
- net LIOD_TX: now reaches CN1_L.27 (Pin_27), CN6_L.1 (Pin_1)
- net LIOD_RX: now reaches CN1_L.14 (Pin_14), CN6_L.2 (Pin_2)
- net LIOD_DET: now reaches CN1_L.25 (Pin_25), CN6_L.3 (Pin_3)
Other:
- note added: ""Coin tray present" switch"
- note added: ""External safe open" switch"
- note added: ""Phone open" switch"
- note removed: "Hookswitch"
- moved on the sheet: C16, C17, CN6, R32, R33, R40, R41, T11
