File: schematics/Rotor_kicad/frontpanel.kicad_sch (KiCad schematic)
At the start: 0 parts

Commit message: Fixed mistakes in main board schematics
Parts:
- added CN2B1: Front panel, symbol Connector_Generic:Conn_02x08_Counter_Clockwise
- added SW12: 1, symbol Switch:SW_Push
- added SW13: 4, symbol Switch:SW_Push
- added SW14: 7, symbol Switch:SW_Push
- added SW15: *, symbol Switch:SW_Push
- added SW16: 2, symbol Switch:SW_Push
- added SW17: 5, symbol Switch:SW_Push
- added SW18: 8, symbol Switch:SW_Push
- added SW19: 0, symbol Switch:SW_Push
- added SW20: 3, symbol Switch:SW_Push
- added SW21: 6, symbol Switch:SW_Push
- added SW22: 9, symbol Switch:SW_Push
- added SW23: #, symbol Switch:SW_Push
- added SWH1: Hookswitch, symbol Switch:SW_Push_DPDT
- added SWR1: Redial button, symbol Switch:SW_SPDT
Connections:
- new net: CN2B1.7 (Pin_7), SWR1.2 (B)
- new net: CN2B1.11 (Pin_11), SWR1.3 (C)
- new net: CN2B1.1 (Pin_1), SWH1.1 (A)
- new net: CN2B1.10 (Pin_10), SWH1.5 (B)
- new net: CN2B1.16 (Pin_16), SWH1.2 (B)
- new net: CN2B1.2 (Pin_2), SWH1.3 (C)
- new net: CN2B1.8 (Pin_8), SWH1.6 (C)
- new net KBD_1: SW13.2, SW17.2, SW21.2
- new net KBD_2: SW14.2, SW18.2, SW22.2
- new net KBD_3: SW20.1, SW21.1, SW22.1, SW23.1
- new net KBD_4: SW15.2, SW19.2, SW23.2
- new net KBD_5: SW12.1, SW13.1, SW14.1, SW15.1
- new net KBD_6: SW12.2, SW16.2, SW20.2
- new net KBD_7: SW16.1, SW17.1, SW18.1, SW19.1
