File: schematics/Rotor_kicad/lcd.kicad_sch (KiCad schematic)
At the start: 0 parts

Commit message: Fixed mistakes in main board schematics
Parts:
- added CN_LCD3: Hitachi LM039 LCD module, symbol Connector_Generic:Conn_02x05_Odd_Even
- added CN_LCD4: LCD module cable connector, symbol Connector_Generic:Conn_02x07_Counter_Clockwise
- added DL3: F.S. LED, symbol Device:LED
- added PM3: LCD contrast, symbol Device:R_Potentiometer_Trim
- added R87: 1M, symbol Device:R
- added R88: 10K, symbol Device:R
- added R89: 150, symbol Device:R
- added SW24: Left, symbol Switch:SW_DIP_x01
- added SW25: RESET, symbol Switch:SW_Push
- added SW26: Right, symbol Switch:SW_DIP_x01
Connections:
- new net: CN_LCD3.10 (Pin_10), CN_LCD4.6 (Pin_6), DL3.2 (A)
- new net: CN_LCD4.1 (Pin_1), SW25.1
- new net: CN_LCD4.7 (Pin_7), SW26.2
- new net: CN_LCD4.8 (Pin_8), SW24.1
- new net: DL3.1 (K), R89.1
- new net +5V: CN_LCD3.2 (Pin_2), CN_LCD4.2 (Pin_2), R87.1, R88.1
- new net CLOCK: CN_LCD3.4 (Pin_4), CN_LCD4.3 (Pin_3)
- new net C/~{D}: CN_LCD3.8 (Pin_8), CN_LCD4.5 (Pin_5)
- new net DATA: CN_LCD3.5 (Pin_5), CN_LCD4.11 (Pin_11)
- new net GND: CN_LCD3.1 (Pin_1), CN_LCD4.13 (Pin_13), CN_LCD4.14 (Pin_14), PM3.1, PM3.2, PM3.3, R89.2, SW24.2, SW25.2, SW26.1
- new net V0: CN_LCD3.3 (Pin_3), CN_LCD4.12 (Pin_12)
- new net ~{BUSY}: CN_LCD3.7 (Pin_7), CN_LCD4.10 (Pin_10), R88.2
- new net ~{CS}: CN_LCD3.6 (Pin_6), CN_LCD4.4 (Pin_4)
- new net ~{RST}: CN_LCD3.9 (Pin_9), CN_LCD4.9 (Pin_9), R87.2
Other:
- note added: "Mode switches: Both ON/Both OFF -> Normal mode SW1 ON, SW2 OFF -> Config mode SW1 OFF, SW2 ON -> Test mode"
- note added: "Stacked w/the cable connector"
