File: schematics/Rotor_kicad/main.kicad_sch (KiCad schematic)
At the start: 117 parts, among them CN1 ., CN2 Front panel, CN3 Headset, CN4 Battery, CN5 Coin tray, CN6 Ext safe?, CN6 LIOD, T1 BC327, T10 BC327, T11 BC237, T12 BC237, T2 MPSA42, T3 MPSA92, T5 MPSA42, T6 MPSA42, T7 MPSA42, T8 MPSA42, T9 BU806, U1 LS358B, U2 ICL7665

Commit message: new schmatics
Parts:
- removed C1: 1 uF, symbol Device:C
- removed C10: 10u 50V, symbol Device:C_Polarized
- removed C11: 300n, symbol Device:C
- removed C12, C16, C17, C3: 1u, symbol Device:C
- removed C13: 10n, symbol Device:C
- removed C14: 470p, symbol Device:C
- removed C15: 220u 100V, symbol Device:C_Polarized
- removed C18, C4, C8: 100n, symbol Device:C
- removed C2: 4.7n, symbol Device:C
- removed C20: 100u 100V, symbol Device:C_Polarized
- removed C6, C7: 22u 50V, symbol Device:C_Polarized
- removed C9: 150n, symbol Device:C
- removed CN1: ., symbol Connector_Generic:Conn_02x20_Counter_Clockwise
- removed CN2: Front panel, symbol Connector_Generic:Conn_02x08_Counter_Clockwise
- removed CN3: Headset, symbol Connector:6P4C
- removed CN4: Battery, symbol Connector:Screw_Terminal_01x02
- removed CN5: Coin tray, symbol Connector_Generic:Conn_01x04
- removed CN6: Ext safe?, symbol Connector_Generic:Conn_01x06
- removed CN6: LIOD, symbol Connector_Generic:Conn_02x06_Counter_Clockwise
- removed D1: "1FK", symbol Simulation_SPICE:DIODE
- removed D10, D11, D12, D13, D14, D15, D2, D4, D5, D6, D7, D8, D9: 1N4007, Diode_THT:D_DO-41_SOD81_P10.16mm_Horizontal, symbol Diode:1N4007
- removed DL1, DL2: LED, symbol Device:LED
- removed DZ1, DZ4: ., symbol Device:D_Zener
- removed DZ2, DZ5: 2.7V, symbol Device:D_Zener
- removed DZ3: 18V, symbol Device:D_Zener
- removed DZ5: 8.2V, symbol Device:D_Zener
- removed DZ6: 1N5988, symbol Device:D_Zener
- removed F5: Fuse, symbol Device:Fuse
- removed ML1: 64357/A, symbol IPM_custom:64357/A
- removed MR1: ., symbol Connector:Screw_Terminal_01x09
- removed OP1, OP2, OP3, OP4: CNY17-1, symbol Isolator:CNY17-1
- removed PM1: 4.7K, symbol Device:R_Potentiometer_Trim
- removed PM2: 100K, symbol Device:R_Potentiometer_Trim
- removed PTC1, PTC2, PTC3, PTC4: ., symbol Device:Thermistor_PTC
- removed R10, R25, R27, R28, R34, R44: 100K, symbol Device:R
- removed R11: 40, symbol Device:R
- removed R12: 8.3K 1%, symbol Device:R
- removed R12: 390, symbol Device:R
- removed R13, R14: 122 1%, symbol Device:R
- removed R15: 2.2K 1%, symbol Device:R
- removed R16: 4.7K, symbol Device:R
- removed R17: 620K 1%, symbol Device:R
- removed R18: 33, symbol Device:R
- removed R19: 13K, symbol Device:R
- removed R23, R24, R38: 150K, symbol Device:R
- removed R26, R40, R5, R7, R9: 10K, symbol Device:R
- removed R29, R3, R30, R32, R33, R39, R4: 100, symbol Device:R
- removed R31, R41, R6: 2.2K, symbol Device:R
- removed R35: 1K, symbol Device:R
- removed R36: 6.8K, symbol Device:R
- removed R37: 300K, symbol Device:R
- removed R42: 3.3K, symbol Device:R
- removed R43: 46K, symbol Device:R
- removed R8: 120K, symbol Device:R
- removed RL1, RL2: SIEMENS-V23042-B2201-B101, symbol Relay:SIEMENS-V23042-B2201-B101
- removed T1, T10: BC327, Package_TO_SOT_THT:TO-92_Inline, symbol Transistor_BJT:BC327
- removed T11, T12: BC237, Package_TO_SOT_THT:TO-92_Inline, symbol Transistor_BJT:BC237
- removed T2, T5, T6, T7, T8, T?: MPSA42, Package_TO_SOT_THT:TO-92_Inline, symbol Transistor_BJT:MPSA42
- removed T3: MPSA92, Package_TO_SOT_THT:TO-92_Inline, symbol Transistor_BJT:MPSA92
- removed T9: BU806, symbol Device:Q_NPN_BCE
- removed U1: LS358B, symbol Interface_Telecom:LS358B
- removed U2: ICL7665, symbol Power_Supervisor:ICL7665
Other:
- note removed: "6V lead acid (charged to 6.75)"
- note removed: "Connectors"
- note removed: "Data comm. line (Power is derived from here)"
- note removed: "Main terminal strip"
- note removed: "Might be a zener"
- note removed: "On some boards, replaced by IC (PT1)"
- note removed: "On some boards, single IC (PT2)"
- note removed: "Pin numbering on silkscreen doesn't match schematic"
- note removed: "Power monitoring"
- note removed: "Power regulation"
- note removed: "Voice circuit"

Commit message: Fixed mistakes in main board schematics
Parts:
- added C49: 470p, symbol Device:C
- added C50: 220u 100V, symbol Device:C_Polarized
- added C51: 100u 100V, symbol Device:C_Polarized
- added C52: 1 uF, symbol Device:C
- added C53, C56, C61: 100n, symbol Device:C
- added C54: 300n, symbol Device:C
- added C55: 10u 50V, symbol Device:C_Polarized
- added C57: 4.7n, symbol Device:C
- added C58: 150n, symbol Device:C
- added C59, C60, C65, C66: 1u, symbol Device:C
- added C62: 10n, symbol Device:C
- added C63, C64: 22u 50V, symbol Device:C_Polarized
- added CN1_L1: ., symbol Connector_Generic:Conn_02x20_Counter_Clockwise
- added CN2_L1: Front panel, symbol Connector_Generic:Conn_02x08_Counter_Clockwise
- added CN3_L1: Headset, symbol Connector:6P4C
- added CN5_L1: Coin tray, symbol Connector_Generic:Conn_01x04
- added CN6_L1: LIOD, symbol Connector_Generic:Conn_02x06_Counter_Clockwise
- added CN7: Battery, symbol Connector:Screw_Terminal_01x02
- added CN8: Ext safe, symbol Connector_Generic:Conn_01x06
- added D37, D38, D39, D40, D41, D42, D43, D44, D45, D47, D48, D49, D50: 1N4007, Diode_THT:D_DO-41_SOD81_P10.16mm_Horizontal, symbol Diode:1N4007
- added D46: 1FK, symbol Simulation_SPICE:DIODE
- added DL4, DL5: LED, symbol Device:LED
- added DZ10: 8.2V, symbol Device:D_Zener
- added DZ11, DZ8: 2.7V, symbol Device:D_Zener
- added DZ12, DZ7: ., symbol Device:D_Zener
- added DZ13: 18V, symbol Device:D_Zener
- added DZ9: 1N5988, symbol Device:D_Zener
- added F1: Fuse, symbol Device:Fuse
- added ML2: 64357/A, symbol IPM_custom:64357/A
- added MR2: ., symbol Connector:Screw_Terminal_01x09
- added OP5, OP6, OP7, OP8: CNY17-1, symbol Isolator:CNY17-1
- added PM4: 4.7K, symbol Device:R_Potentiometer_Trim
- added PM5: 100K, symbol Device:R_Potentiometer_Trim
- added PTC5, PTC6, PTC7, PTC8: ., symbol Device:Thermistor_PTC
- added R186: 3.3K, symbol Device:R
- added R187, R197, R222: 2.2K, symbol Device:R
- added R188, R198, R202, R204, R221: 10K, symbol Device:R
- added R189, R194, R201, R203, R220, R223, R224: 100, symbol Device:R
- added R190, R192, R196, R199, R215, R225: 100K, symbol Device:R
- added R191, R193, R212: 150K, symbol Device:R
- added R195: 46K, symbol Device:R
- added R200: 120K, symbol Device:R
- added R205: 1K, symbol Device:R
- added R206: 6.8K, symbol Device:R
- added R207: 13K, symbol Device:R
- added R208: 33, symbol Device:R
- added R209: 4.7K, symbol Device:R
- added R210: 40, symbol Device:R
- added R211: 300K, symbol Device:R
- added R213: 620K 1%, symbol Device:R
- added R214: 390, symbol Device:R
- added R216: 8.3K 1%, symbol Device:R
- added R217, R219: 122 1%, symbol Device:R
- added R218: 2.2K 1%, symbol Device:R
- added RL3, RL4: SIEMENS-V23042-B2201-B101, symbol Relay:SIEMENS-V23042-B2201-B101
- added T19, T21, T22, T23, T26, T27: MPSA42, Package_TO_SOT_THT:TO-92_Inline, symbol Transistor_BJT:MPSA42
- added T20: BU806, symbol Device:Q_NPN_BCE
- added T24, T30: BC237, Package_TO_SOT_THT:TO-92_Inline, symbol Transistor_BJT:BC237
- added T25, T29: BC327, Package_TO_SOT_THT:TO-92_Inline, symbol Transistor_BJT:BC327
- added T28: MPSA92, Package_TO_SOT_THT:TO-92_Inline, symbol Transistor_BJT:MPSA92
- added U28: ICL7665, symbol Power_Supervisor:ICL7665
- added U29: LS358B, symbol Interface_Telecom:LS358B
Connections:
- new net: R199.1, U28.3 (SET1)
- new net: C58.2, C60.1, R213.1, U29.16 (MIC_IN)
- new net: C54.1, C55.2, C57.1, C60.2, C62.1, CN3_L1.4, D49.2 (A), D50.2 (A), DZ13.2 (A), R207.2, R208.1, R215.1, R216.2, RL3.7 (11), U29.3 (MUTING), U29.9 (LINE_-)
- new net: C57.2, C59.2, C61.1, DZ13.1 (K), OP8.4, R202.2, R210.2, RL3.8 (13), T26.1 (E), T27.1 (E), U29.2 (LINE_+)
- new net: D42.2 (A), DZ7.1 (K), DZ8.2 (A), PTC6.2
- new net: D38.2 (A), D40.1 (K), DZ7.2 (A), OP6.2, PTC5.2
- new net: C53.1, R205.1, R206.2, T29.2 (B)
- new net: R205.2, U28.7 (OUT2)
- new net: D44.1 (K), D45.2 (A)
- new net: D43.1 (K), D44.2 (A)
- new net: D37.2 (A), OP5.4, R187.2, R188.1, R190.1, R192.1, T22.1 (E), T23.3 (C)
- new net: R190.2, T19.1 (E), T21.2 (B)
- new net: C52.1, R203.1
- new net: C52.2, D48.2 (A), D50.1 (K), RL4.6 (9)
- new net: MR2.9 (Pin_9), PTC5.1
- new net: MR2.8 (Pin_8), PTC6.1
- new net: D47.1 (K), D48.1 (K), DZ11.1 (K), R201.1
- new net: C50.2, D40.2 (A), D41.2 (A), DL5.1 (K), DZ9.2 (A), R186.1, R194.2
- new net: OP6.1, R193.2
- new net: C56.2, C58.1, R213.2, U29.1 (MIC_IN)
- new net: C61.2, R214.1, R218.1, U29.10 (INPUT_-)
- new net: C59.1, U29.11 (INPUT_+)
- new net: R217.2, U29.12 (REC_OUT)
- new net: R219.2, U29.13 (REC_OUT)
- new net: R215.2, U29.14 (MF_INPUT)
- new net: R207.1, U29.4 (BIAS_ADJ)
- new net: C55.1, U29.5 (SHUNT_BYPASS), U29.8 (GAIN_CTRL)
- new net: R210.1, R214.2, U29.6 (DC_REG)
- new net: R208.2, U29.7 (CURR_SENSE)
- new net: OP7.1, R201.2
- new net: DZ11.2 (A), OP7.2, R200.2, R204.1, RL3.6 (9), T26.3 (C), T28.1 (E)
- new net: OP7.5, R198.2
- new net: C49.1, OP5.5, R191.1, T19.2 (B)
- new net: R188.2, T21.1 (E), T22.2 (B)
- new net: PM4.3, R186.2, T20.1 (B)
- new net: R187.1, T20.2 (C)
- new net: R202.1, T26.2 (B), T28.3 (C)
- new net: CN1_L1.17 (Pin_17), T30.1 (C)
- new net: R221.2, R222.1, T30.2 (B)
- new net: CN2_L1.10 (Pin_10), R221.1
- new net: D46.1 (A), OP8.5, R200.1
- new net: ML2.4 (I_LIMIT), R195.1
- new net: R195.2, R196.1, T24.2 (B)
- new net: CN1_L1.27 (Pin_27), CN6_L1.1 (Pin_1)
- new net: CN1_L1.34 (Pin_34), CN6_L1.10 (Pin_10)
- new net: CN1_L1.14 (Pin_14), CN6_L1.2 (Pin_2)
- new net: CN1_L1.25 (Pin_25), CN6_L1.3 (Pin_3)
- new net: CN1_L1.18 (Pin_18), CN6_L1.4 (Pin_4)
- new net: CN6_L1.5 (Pin_5), R225.2
- new net: CN8.1 (Pin_1), R223.2
- new net: C62.2, R216.1, R218.2
- new net: DZ12.2 (A), PTC7.2, R203.2, RL4.8 (13)
- new net: D46.2 (K), T27.2 (B)
- new net: DL4.2 (A), R192.2, T23.2 (B)
- new net: PM5.1, R212.1
- new net: PM5.2, U28.5 (SET2)
- new net: PM5.3, R211.2
- new net: D47.2 (A), D49.1 (K), DZ12.1 (K), PTC8.2
- new net: D39.2 (A), D41.1 (K), D42.1 (K), DZ8.1 (K), R193.1
- new net: CN1_L1.10 (Pin_10), CN5_L1.4 (Pin_4)
- new net: CN1_L1.22 (Pin_22), CN8.5 (Pin_5)
- new net: CN1_L1.24 (Pin_24), R220.1
- new net: CN1_L1.32 (Pin_32), CN5_L1.2 (Pin_2)
- new net: CN1_L1.36 (Pin_36), CN2_L1.9 (Pin_9)
- new net: CN1_L1.5 (Pin_5), CN2_L1.11 (Pin_11)
- new net: CN7.2 (Pin_2), F1.1
- new net: R204.2, T27.3 (C), T28.2 (B)
- new net: DL4.1 (K), DL5.2 (A)
- new net: PM4.1, PM4.2, R189.1
- new net: R189.2, T23.1 (E)
- new net: C63.1, C64.1
- new net: C63.2, R217.1
- new net: C56.1, CN3_L1.3, R209.2
- new net: CN8.2 (Pin_2), CN8.4 (Pin_4), R224.1
- new net: CN2_L1.1 (Pin_1), MR2.2 (Pin_2)
- new net: CN2_L1.16 (Pin_16), MR2.3 (Pin_3)
- new net: CN2_L1.2 (Pin_2), MR2.1 (Pin_1)
- new net: CN2_L1.7 (Pin_7), R220.2
- new net: R197.2, R198.1, T25.2 (B)
- new net: C64.2, CN3_L1.1
- new net: MR2.6 (Pin_6), PTC8.1
- new net: MR2.7 (Pin_7), PTC7.1
- new net: MR2.4 (Pin_4), RL4.7 (11)
- new net: CN3_L1.2, R219.1
- new net +5V: CN1_L1.12 (Pin_12), CN1_L1.15 (Pin_15), CN1_L1.29 (Pin_29), CN2_L1.6 (Pin_6), CN2_L1.8 (Pin_8), CN5_L1.1 (Pin_1), CN5_L1.3 (Pin_3), CN6_L1.8 (Pin_8), CN8.6 (Pin_6), D45.1 (K), R197.1, R211.1, RL4.10 (16), RL4.9 (15), T25.3 (E), T29.1 (C)
- new net +BATT: C51.1, C53.2, CN1_L1.13 (Pin_13), CN1_L1.28 (Pin_28), CN6_L1.7 (Pin_7), D43.2 (A), DZ10.1 (K), F1.2, ML2.5 (BATTERY), R199.2, R206.1, T29.3 (E), U28.8 (V+)
- new net AC_DIN: CN1_L1.31 (Pin_31), T25.1 (C)
- new net AC_DOUT: CN1_L1.9 (Pin_9), OP8.1
- new net AS_BRIDGE_+: C49.2, D38.1 (K), D39.1 (K), R191.2, R225.1, T19.3 (C), T21.3 (C), T22.3 (C)
- new net AS_DIN: CN1_L1.33 (Pin_33), OP6.5
- new net AS_DOUT: CN1_L1.8 (Pin_8), OP5.1
- new net GND: C51.2, C65.1, C66.1, CN1_L1.11 (Pin_11), CN1_L1.30 (Pin_30), CN6_L1.11 (Pin_11), CN6_L1.12 (Pin_12), CN6_L1.9 (Pin_9), CN7.1 (Pin_1), CN8.3 (Pin_3), DZ10.2 (A), DZ9.1 (K), ML2. (GND), ML2.2 (GND), OP5.2, OP6.4, OP7.4, OP8.2, R194.1, R196.2, R212.2, R222.2, RL3.10 (16), RL3.9 (15), T20.3 (E), T24.3 (E), T30.3 (E), U28.4 (GND)
- new net KBD_1: CN1_L1.2 (Pin_2), CN2_L1.15 (Pin_15)
- new net KBD_2: CN1_L1.1 (Pin_1), CN2_L1.3 (Pin_3)
- new net KBD_3: CN1_L1.40 (Pin_40), CN2_L1.14 (Pin_14)
- new net KBD_4: CN1_L1.39 (Pin_39), CN2_L1.4 (Pin_4)
- new net KBD_5: CN1_L1.3 (Pin_3), CN2_L1.13 (Pin_13)
- new net KBD_6: CN1_L1.38 (Pin_38), CN2_L1.5 (Pin_5)
- new net KBD_7: CN1_L1.4 (Pin_4), CN2_L1.12 (Pin_12)
- new net LINE: C50.1, CN6_L1.6 (Pin_6), D37.1 (K), ML2.1 (LINE)
- new net RL1-R: CN1_L1.6 (Pin_6), RL4.1
- new net RL1-S: CN1_L1.37 (Pin_37), RL4.2
- new net RL2-R: CN1_L1.7 (Pin_7), RL3.1
- new net RL2-S: CN1_L1.35 (Pin_35), RL3.2
- new net SAFE_SW1: C65.2, CN1_L1.19 (Pin_19), R223.1
- new net SAFE_SW2: C66.2, CN1_L1.20 (Pin_20), R224.2
- new net VDD: C54.2, R209.1, U29.15 (VDD)
- new net ~{I_LIMIT}: CN1_L1.26 (Pin_26), T24.1 (C)
- no-connect marks 0 -> 3
Other:
- note added: "6V lead acid (charged to 6.75)"
- note added: "Connectors"
- note added: "Data comm. line (Power is derived from here)"
- note added: "Main terminal strip"
- note added: "Might be a zener"
- note added: "On some boards, replaced by IC (PT1)"
- note added: "On some boards, single IC (PT2)"
- note added: "Pin numbering on silkscreen doesn't match schematic"
- note added: "Power monitoring"
- note added: "Power regulation"
- note added: "Voice circuit"
