File: schematics/Rotor_kicad/modules_67381.kicad_sch (KiCad schematic)
At the start: 0 parts

Commit message: Fixed mistakes in main board schematics
Parts:
- added C39, C40, C41: 150n, symbol Device:C
- added J6: ., symbol Connector:Conn_01x13_Male
- added Q26, Q27: BC847, Package_TO_SOT_SMD:SOT-23, symbol Transistor_BJT:BC847
- added R141, R142, R143, R144, R145, R146, R147, R148, R149, R150: 100K, symbol Device:R
- added U24: 40106, symbol 4xxx:40106
Connections:
- new net: C41.2, R146.1, U24.3
- new net: J6.3 (Pin_3), R141.2, R146.2
- new net: J6.7 (Pin_7), U24.12, U24.5
- new net: J6.8 (Pin_8), U24.6
- new net: C40.2, R145.1, U24.13
- new net: J6.2 (Pin_2), R142.2, R145.2
- new net: R147.1, U24.8
- new net: Q27.1 (B), R147.2, R148.1
- new net: Q26.1 (B), R149.2, R150.1
- new net: C39.2, R144.2, U24.1
- new net: J6.5 (Pin_5), U24.2
- new net: J6.6 (Pin_6), U24.4
- new net: R149.1, U24.10
- new net: J6.9 (Pin_9), U24.11
- new net: J6.1 (Pin_1), R143.2, R144.1
- new net: J6.10 (Pin_10), U24.9
- new net: J6.11 (Pin_11), Q26.3 (C)
- new net: J6.13 (Pin_13), Q27.3 (C)
- new net +5V: J6.4 (Pin_4), U24.14 (VDD)
- new net GND: C39.1, C40.1, C41.1, J6.12 (Pin_12), Q26.2 (E), Q27.2 (E), R141.1, R142.1, R143.1, R148.2, R150.2, U24.7 (VSS)
Other:
- note added: "No designators present on module. Resistors are thick-film on ceramic, laser trimmed. Reported values are direct measures."
