File: schematics/Rotor_kicad/modules_67382.kicad_sch (KiCad schematic)
At the start: 0 parts

Commit message: Fixed mistakes in main board schematics
Parts:
- added J5: ., symbol Connector:Conn_01x10_Male
- added Q22, Q23, Q24, Q25: BC857, Package_TO_SOT_SMD:SOT-23, symbol Transistor_BJT:BC857
- added R130, R132, R136: ?, symbol Device:R
- added R131, R134, R137: 3.3K, symbol Device:R
- added R133, R135, R138: 1.6K, symbol Device:R
- added R139, R140: 45K, symbol Device:R
- added U23: 74HC14, symbol 74xx:74HC14
Connections:
- new net: Q24.1 (B), R137.1, R138.2
- new net: Q25.3 (C), R140.1, U23.13
- new net: J5.3 (Pin_3), R132.2, R134.2
- new net: J5.10 (Pin_10), Q25.1 (B)
- new net: Q23.1 (B), R134.1, R135.2
- new net: Q23.3 (C), U23.5
- new net: Q22.3 (C), U23.1
- new net: J5.2 (Pin_2), U23.2
- new net: J5.1 (Pin_1), R130.2, R131.2
- new net: J5.4 (Pin_4), U23.6
- new net: J5.6 (Pin_6), U23.12
- new net: J5.7 (Pin_7), U23.8
- new net: J5.8 (Pin_8), R136.2, R137.2
- new net: Q24.3 (C), R139.1, U23.9
- new net: Q22.1 (B), R131.1, R133.2
- new net +5V: J5.9 (Pin_9), Q22.2 (E), Q23.2 (E), Q24.2 (E), Q25.2 (E), R130.1, R132.1, R133.1, R135.1, R136.1, R138.1
- new net GND: J5.5 (Pin_5), R139.2, R140.2, U23.11, U23.3
Other:
- note added: "No designators present on module. Resistors are thick-film on ceramic, laser trimmed. Reported values are direct measures."
