File: schematics/Rotor_kicad/modules_67383.kicad_sch (KiCad schematic)
At the start: 0 parts

Commit message: Fixed mistakes in main board schematics
Parts:
- added C42, C43, C44: C, symbol Device:C
- added J8: ., symbol Connector:Conn_01x10_Male
- added Q35: BC847, Package_TO_SOT_SMD:SOT-23, symbol Transistor_BJT:BC847
- added Q36: BCW67, Package_TO_SOT_SMD:SOT-23, symbol Transistor_BJT:BC857
- added R170: 20.5K, symbol Device:R
- added R171: 100K, symbol Device:R
- added R172: 3.3K, symbol Device:R
- added R173, R174: 32K, symbol Device:R
- added R175: 260, symbol Device:R
- added R176: 1K, symbol Device:R
- added U25: HEF4093B, symbol 4xxx:HEF4093B
Connections:
- new net: J8.1 (Pin_1), R171.2, U25.1, U25.12
- new net: C43.1, J8.7 (Pin_7), R172.2, U25.13
- new net: C43.2, J8.6 (Pin_6), U25.10
- new net: U25.11, U25.5
- new net: J8.3 (Pin_3), R170.1, U25.3, U25.8, U25.9
- new net: C42.1, J8.2 (Pin_2), R170.2, U25.2
- new net: C44.2, Q35.1 (B), R175.1, R176.2
- new net: J8.9 (Pin_9), Q35.3 (C)
- new net: R173.1, U25.4
- new net: Q36.1 (B), R173.2, R174.1
- new net: C44.1, Q36.3 (C), R175.2
- new net: J8.4 (Pin_4), U25.6
- new net +5V: J8.8 (Pin_8), Q36.2 (E), R172.1, R174.2, U25.14 (VCC)
- new net GND: C42.2, J8.10 (Pin_10), J8.5 (Pin_5), Q35.2 (E), R171.1, R176.1, U25.7 (GND)
Other:
- note added: "No designators present on module. Resistors are thick-film on ceramic, laser trimmed. Reported values are direct measures."
