File: schematics/Rotor_kicad/modules_67384.kicad_sch (KiCad schematic)
At the start: 0 parts

Commit message: Fixed mistakes in main board schematics
Parts:
- added D29, D30, D31, D32: ?, Diode_THT:D_DO-41_SOD81_P10.16mm_Horizontal, symbol Diode:1N4007
- added J4: ., symbol Connector:Conn_01x20_Male
- added Q12, Q13, Q16, Q18, Q20, Q21: BC847, Package_TO_SOT_SMD:SOT-23, symbol Transistor_BJT:BC847
- added Q14, Q15, Q17, Q19: BC857, Package_TO_SOT_SMD:SOT-23, symbol Transistor_BJT:BC857
- added R114, R115, R120, R121, R128, R129: 6.5K, symbol Device:R
- added R116, R117: 210, symbol Device:R
- added R118: 100, symbol Device:R
- added R119: 10, symbol Device:R
- added R122, R127: 330, symbol Device:R
- added R123, R124, R125, R126: 220, symbol Device:R
- added U22: 4001, symbol 4xxx:4001
Connections:
- new net: Q15.1 (B), R118.2, R119.1
- new net: Q13.3 (C), R119.2
- new net: J4.3 (Pin_3), Q13.1 (B), U22.12
- new net: Q17.1 (B), R124.1, R127.1
- new net: D29.1 (K), D31.1 (K), Q14.3 (C), Q15.2 (E), Q17.2 (E), Q19.2 (E), R118.1, R124.2, R125.2
- new net: D29.2 (A), D30.1 (K), J4.12 (Pin_12), Q17.3 (C), Q18.3 (C)
- new net: Q16.2 (E), Q18.1 (B), R123.2
- new net: Q16.1 (B), R120.2, R121.1
- new net: Q16.3 (C), R122.2
- new net: Q21.1 (B), R128.1, R129.1
- new net: Q19.1 (B), R122.1, R125.1
- new net: Q14.1 (B), R116.2, R117.1
- new net: Q21.3 (C), R127.2
- new net: Q20.1 (B), Q21.2 (E), R126.2
- new net: R120.1, U22.4
- new net: D31.2 (A), D32.1 (K), J4.18 (Pin_18), Q19.3 (C), Q20.3 (C)
- new net: Q12.1 (B), R114.2, R115.1
- new net: Q12.3 (C), R117.2
- new net: R129.2, U22.10, U22.6
- new net: J4.5 (Pin_5), U22.8
- new net: U22.13, U22.3, U22.5, U22.9
- new net: J4.7 (Pin_7), U22.1, U22.2
- new net: R114.1, U22.11
- new net +5V: J4.4 (Pin_4), U22.14 (VDD)
- new net +BATT: J4.15 (Pin_15), J4.16 (Pin_16), Q14.2 (E), R116.1
- new net GND: D30.2 (A), D32.2 (A), J4.1 (Pin_1), J4.10 (Pin_10), J4.11 (Pin_11), J4.17 (Pin_17), J4.2 (Pin_2), J4.20 (Pin_20), J4.6 (Pin_6), J4.8 (Pin_8), J4.9 (Pin_9), Q12.2 (E), Q13.2 (E), Q15.3 (C), Q18.2 (E), Q20.2 (E), R115.2, R121.2, R123.1, R126.1, R128.2, U22.7 (VSS)
- no-connect marks 0 -> 3
Other:
- note added: "No designators present on module. Resistor are thick-film on ceramic, laser trimmed. Reported values are direct measures."
