File: schematics/Rotor_kicad/modules_67475.kicad_sch (KiCad schematic)
At the start: 0 parts

Commit message: Fixed mistakes in main board schematics
Parts:
- added J7: ., symbol Connector:Conn_01x15_Male
- added Q28, Q29, Q30, Q31, Q32, Q33: BCW67, Package_TO_SOT_SMD:SOT-23, symbol Transistor_BJT:BC857
- added Q34: BC847, Package_TO_SOT_SMD:SOT-23, symbol Transistor_BJT:BC847
- added R151, R154, R157, R160, R163: 1K, symbol Device:R
- added R152, R153, R155, R156, R158, R159, R161, R162, R164, R165, R166, R167: 10K, symbol Device:R
- added R168, R169: 100K, symbol Device:R
Connections:
- new net: J7.9 (Pin_9), Q28.2 (E), Q29.2 (E), Q30.2 (E), Q31.2 (E), Q32.2 (E), R152.1, R155.1, R158.1, R161.1, R164.1
- new net: Q31.1 (B), R161.2, R162.1
- new net: Q30.1 (B), R158.2, R159.1
- new net: Q30.3 (C), R157.1
- new net: Q32.1 (B), R164.2, R165.1
- new net: J7.11 (Pin_11), R165.2
- new net: J7.5 (Pin_5), R157.2
- new net: Q29.1 (B), R155.2, R156.1
- new net: Q28.1 (B), R152.2, R153.1
- new net: J7.2 (Pin_2), R153.2
- new net: J7.4 (Pin_4), R156.2
- new net: Q29.3 (C), R154.1
- new net: J7.3 (Pin_3), R154.2
- new net: J7.12 (Pin_12), Q33.2 (E), R166.1
- new net: Q33.1 (B), R166.2, R167.1
- new net: J7.8 (Pin_8), R162.2
- new net: J7.14 (Pin_14), Q34.2 (E), R168.1
- new net: Q34.1 (B), R168.2, R169.2
- new net: Q34.3 (C), R167.2
- new net: Q31.3 (C), R160.1
- new net: J7.13 (Pin_13), Q33.3 (C)
- new net: Q28.3 (C), R151.1
- new net: Q32.3 (C), R163.1
- new net: J7.10 (Pin_10), R163.2
- new net: J7.15 (Pin_15), R169.1
- new net: J7.7 (Pin_7), R160.2
- new net: J7.1 (Pin_1), R151.2
- new net: J7.6 (Pin_6), R159.2
Other:
- note added: "No designators present on module. Resistors are thick-film on ceramic, laser trimmed. Reported values are direct measures."
