File: schematics/Rotor_kicad/modules_67476.kicad_sch (KiCad schematic)
At the start: 0 parts

Commit message: Fixed mistakes in main board schematics
Parts:
- added C45, C46, C47, C48: 100n, symbol Device:C
- added D33: "225", Package_TO_SOT_SMD:SOT-323_SC-70, symbol Diode:BAS16W
- added D34, D35, D36: BAS16W, Package_TO_SOT_SMD:SOT-323_SC-70, symbol Diode:BAS16W
- added J9: ~, symbol Connector:Conn_01x15_Pin
- added Q37: Si2301, Package_TO_SOT_SMD:SOT-23, symbol Transistor_FET:Si2319CDS
- added R177: 20.8k, symbol Device:R
- added R178: 170k, symbol Device:R
- added R179, R180: 100k, symbol Device:R
- added R181: 11.6k, symbol Device:R
- added R182, R184, R185: 10k, symbol Device:R
- added R183: 100, symbol Device:R
- added U26: HEF4093B, symbol 4xxx:HEF4093B
- added U27: 74HC14, symbol 74xx:74HC14
Connections:
- new net: C46.2, Q37.2 (S), R182.1, U27.9
- new net: J9.4 (Pin_4), R179.2, U26.12
- new net: D34.1 (A), R177.1
- new net: D34.3 (K), U26.1, U26.2, U26.4
- new net: D33.3 (K), R177.2, R178.2, U26.5
- new net: J9.2 (Pin_2), U26.6
- new net: J9.9 (Pin_9), U27.10
- new net: C46.1, U27.11, U27.12
- new net: C48.1, D36.3 (K), R185.1, U27.1
- new net: C47.2, D35.3 (K), R184.2, U27.5
- new net: J9.3 (Pin_3), R178.1, U26.3
- new net: J9.8 (Pin_8), U27.13
- new net: J9.10 (Pin_10), U27.8
- new net: J9.11 (Pin_11), U27.4
- new net: J9.12 (Pin_12), U27.2
- new net: J9.15 (Pin_15), R183.1
- new net: J9.5 (Pin_5), U26.10
- new net: J9.6 (Pin_6), R180.2, U26.13
- new net: C48.2, U27.3, U27.6
- new net: D35.1 (A), R183.2
- new net: C45.2, Q37.1 (G), R181.2, U26.8, U26.9
- new net: C45.1, U26.11
- new net +5V: J9.7 (Pin_7), R179.1, R180.1, U26.14 (VCC), U27.14 (VCC)
- new net GND: C47.1, D33.1 (A), D36.1 (A), J9.1 (Pin_1), J9.14 (Pin_14), Q37.3 (D), R181.1, R182.2, R184.1, R185.2, U26.7 (GND), U27.7 (GND)
- no-connect marks 0 -> 1
Other:
- note added: "No designators present on module. Resistors are thick-film on ceramic, laser trimmed. Reported values are direct measures."
