File: schematics/Rotor_kicad/rotor_main.kicad_sch (KiCad schematic)
At the start: 0 parts

Commit message: Fixed mistakes in main board schematics
Parts:
- added AR1: ~, Resistor_THT:R_Array_SIP9, symbol Device:R_Network08
- added C23, C25, C26, C27, C28, C29, C30, C32, C33, C34, C35, C36: 100n, symbol Device:C
- added C24, C31: ~, symbol Device:C_Polarized
- added CN3: Mechanical section connector, symbol Connector_Generic:Conn_02x30_Counter_Clockwise
- added CN5: Line interface connector, symbol Connector_Generic:Conn_02x20_Counter_Clockwise
- added CNA1, CNB1, CNC1: ~, symbol Connector_Generic:Conn_02x16_Counter_Clockwise
- added CN_COIN1: Coin discriminator module, symbol Connector_Generic:Conn_02x06_Counter_Clockwise
- added CN_LCD1: LCD module cable connector, symbol Connector_Generic:Conn_02x07_Counter_Clockwise
- added D19, D20, D21, D26: 1N4148, Diode_THT:D_DO-35_SOD27_P7.62mm_Horizontal, symbol Diode:1N4148
- added H10: ~, symbol IPM_custom:67384
- added H11, H13: ~, symbol IPM_custom:67381
- added H12: ~, symbol IPM_custom:67475
- added H14: 67382, symbol IPM_custom:67382
- added H15: 67476 hybrid, symbol Connector:Conn_01x15_Pin
- added H16, H17, H18: ~, symbol IPM_custom:67383
- added JP2: ~, symbol Jumper:Jumper_2_Bridged
- added M2: Rotor motor, symbol Motor:Motor_DC
- added OPT5: Rotor pocket exit photointerrupter, OptoDevice:Everlight_ITR9608-F, symbol Sensor_Proximity:ITR9608-F
- added OPT6: Coin tray entrance photointerrupter, OptoDevice:Everlight_ITR9608-F, symbol Sensor_Proximity:ITR9608-F
- added OPT7: "Rotor pocket open" photointerrupter, OptoDevice:Everlight_ITR9608-F, symbol Sensor_Proximity:ITR9608-F
- added OPT8: Rotor pocket entrance photointerrupter, OptoDevice:Everlight_ITR9608-F, symbol Sensor_Proximity:ITR9608-F
- added R6, R71: ~, symbol Device:R
- added R70, R73: 100, symbol Device:R
- added R72, R74, R75, R76, R77, R80, R82: 100k, symbol Device:R
- added R78, R79, R81: 10k, symbol Device:R
- added R83: 1.8k, symbol Device:R
- added R84: 3.9k, symbol Device:R
- added R85: 22k, symbol Device:R
- added R86: 180, symbol Device:R
- added RN2: AR1, Resistor_THT:R_Array_SIP9, symbol Device:R_Network08
- added SOL4: Coin reject solenoid, symbol Device:L_Iron
- added SOL5: Coin path solenoid, symbol Device:L_Iron
- added SOL6: Coin rotor pocket open/close solenoid, symbol Device:L_Iron
- added SW_C_PATH1: Coin path switch, symbol Switch:SW_SPST
- added SW_ENC5, SW_ENC6, SW_ENC7, SW_ENC8, SW_ENC9: Rotor absolute position encoder, symbol Switch:SW_SPST
- added SW_REJ1: Coin reject actuator switch, symbol Switch:SW_SPST
- added U10: 4001, symbol 4xxx:4001
- added U11: 74LS125, symbol 74xx:74LS125
- added U12: 4023, symbol 4xxx:4023
- added U13: 4556, symbol 4xxx_IEEE:4556
- added U14, U15: 74HC244, symbol 74xx:74HC244
- added U16: 74LS148, symbol 74xx:74LS148
- added U17, U18: 74HC373, symbol 74xx:74HC373
Connections:
- new net: H16.4 (IN2), U18.15 (O5)
- new net: H17.4 (IN2), U18.9 (O3)
- new net: OPT6.1, R70.2
- new net: CN3.40 (Pin_40), R73.2
- new net: H11.10 (IN), U11.1, U11.10, U11.13, U11.4, U13.5 (~{Q1})
- new net: U13.6 (~{Q2}), U15.1 (1OE), U15.19 (2OE)
- new net: H11.9 (IN), U13.7 (~{Q3}), U14.1 (1OE), U14.19 (2OE)
- new net: H10.7 (DRV_EN), U10.4
- new net: D21.1 (K), U13.11 (~{Q1})
- new net: H14.4 (OUT), U11.12
- new net: U12.12, U12.6
- new net: H14.10 (IN), R83.2, R84.2
- new net: H14.6 (OUT), U14.15 (2A1)
- new net: U14.6 (1A2), U16.6 (S2)
- new net: U14.4 (1A1), U16.7 (S1)
- new net: U14.2 (1A0), U16.9 (S0)
- new net: H11.7 (OUT1), U15.13 (2A2)
- new net: H14.2 (OUT), U11.5
- new net: H15.12 (Pin_12), U12.3
- new net: H15.10 (Pin_10), U12.4
- new net: H15.5 (Pin_5), U12.5
- new net: H15.4 (Pin_4), JP2.2 (B), R71.2
- new net: D20.1 (K), U13.10 (~{Q2})
- new net: D26.1 (K), U13.12 (~{Q0})
- new net: D19.1 (K), U13.9 (~{Q3})
- new net: H14.7 (OUT), U11.9
- new net: H11.6 (OUT), H16.1 (IN1)
- new net: H13.6 (OUT), U14.17 (2A0)
- new net: U10.10, U10.5
- new net: H12.15 (IN), H15.3 (Pin_3)
- new net: H13.7 (OUT1), U14.13 (2A2)
- new net +5V: AR1.1 (common), C23.2, C25.2, C26.2, C27.2, C28.2, C29.2, C30.2, C31.1, CN3.2 (Pin_2), CN3.43 (Pin_43), CN3.47 (Pin_47), CN3.9 (Pin_9), CN5.12 (Pin_12), CN5.29 (Pin_29), CNA1.16 (Pin_16), CNA1.17 (Pin_17), CNA1.3 (Pin_3), CNA1.30 (Pin_30), CNC1.23 (Pin_23), CN_COIN1.1 (Pin_1), CN_LCD1.2 (Pin_2), H10.4 (VCC), H11.4 (VCC), H13.4 (VCC), H14.9 (VCC), H15.7 (Pin_7), H16.8 (VCC), H17.8 (VCC), H18.8 (VCC), R6.1, R71.1, R74.1, R75.1, R76.1, R77.1, R78.1, R79.1, R80.1, R81.1, R82.1, R83.1, R85.1, RN2.1 (common), SW_C_PATH1.2 (B), SW_REJ1.2 (B), U10.14 (VDD), U11.14 (VCC), U12.14 (VDD), U12.2, U12.8, U13.16 (Vdd), U13.8 (Vss), U14.20 (VCC), U15.20 (VCC), U16.16 (VCC), U17.20 (VCC), U18.20 (VCC)
- new net +BATT: C24.1, CN3.36 (Pin_36), CN3.42 (Pin_42), CN3.44 (Pin_44), CN3.46 (Pin_46), CN5.13 (Pin_13), CN5.28 (Pin_28), H10.15 (VBAT1), H10.16 (VBAT2), H12.13 (VBAT), OPT5.1, R70.1, R73.1, SOL4.2, SOL5.2, SOL6.2
- new net AC_DIN: CN5.31 (Pin_31), R72.1, U12.1
- new net AC_DOUT: CN5.9 (Pin_9), H12.1 (OUT)
- new net AS_DIN: CN5.33 (Pin_33), CNA1.5 (Pin_5), JP2.1 (A), R6.2
- new net AS_DOUT: CN5.8 (Pin_8), H12.3 (OUT)
- new net B_A0: CNB1.21 (Pin_21), U17.3 (D0), U18.3 (D0)
- new net B_A1: CNB1.12 (Pin_12), U17.4 (D1), U18.4 (D1)
- new net B_A2: CNB1.22 (Pin_22), U17.7 (D2), U18.7 (D2)
- new net B_A3: CNB1.11 (Pin_11), U17.8 (D3), U18.8 (D3)
- new net B_A4: CNB1.23 (Pin_23), U17.13 (D4), U18.13 (D4)
- new net B_A5: CNB1.10 (Pin_10), U17.14 (D5), U18.14 (D5)
- new net B_A6: CNB1.24 (Pin_24), U17.17 (D6), U18.17 (D6)
- new net B_A7: CNB1.9 (Pin_9), U17.18 (D7), U18.18 (D7)
- new net CN1-21: CN3.21 (Pin_21), CN3.38 (Pin_38), OPT6.2, OPT7.1
- new net CN1-23: CN3.23 (Pin_23), CN3.31 (Pin_31), OPT7.2, OPT8.1
- new net CN1-53: CN3.53 (Pin_53), CN_COIN1.6 (Pin_6), H15.8 (Pin_8)
- new net CN2-16: CN5.16 (Pin_16), H15.6 (Pin_6)
- new net CN2-18: CN5.18 (Pin_18), CNC1.14 (Pin_14)
- new net CN2-21: U10.12, U10.3
- new net CN2-22: CN5.22 (Pin_22), H11.11 (OUT), R86.2
- new net CN2-34: CN5.34 (Pin_34), H12.5 (OUT)
- new net COIN_D0: CN3.51 (Pin_51), CN_COIN1.5 (Pin_5), U16.5 (EI)
- new net COIN_D1: CN3.48 (Pin_48), CN_COIN1.2 (Pin_2), U16.11 (I1)
- new net COIN_D2: CN3.11 (Pin_11), CN_COIN1.9 (Pin_9), U16.12 (I2)
- new net COIN_D3: CN3.50 (Pin_50), CN_COIN1.4 (Pin_4), U16.13 (I3)
- new net COIN_D4: CN3.12 (Pin_12), CN_COIN1.10 (Pin_10), U16.1 (I4)
- new net COIN_D5: CN3.49 (Pin_49), CN_COIN1.3 (Pin_3), U16.2 (I5)
- new net COIN_D6: CN3.13 (Pin_13), CN_COIN1.11 (Pin_11), U16.3 (I6)
- new net COIN_SW1: CN5.10 (Pin_10), H13.3 (IN)
- new net COIN_SW2: CN5.32 (Pin_32), H13.2 (IN)
- new net C_A0: CNC1.28 (Pin_28), U17.2 (O0)
- new net C_A1: CNC1.7 (Pin_7), U17.5 (O1)
- new net C_A10: CNC1.27 (Pin_27)
- new net C_A2: CNC1.26 (Pin_26), U17.6 (O2)
- new net C_A3: CNC1.8 (Pin_8), U17.9 (O3)
- new net C_A4: CNC1.25 (Pin_25), U17.12 (O4)
- new net C_A5: CNC1.24 (Pin_24), U17.15 (O5)
- new net C_A6: CNC1.10 (Pin_10), U17.16 (O6)
- new net C_A7: CNC1.22 (Pin_22), U17.19 (O7)
- new net C_A8: CNC1.11 (Pin_11), U18.2 (O0)
- new net C_A9: CNC1.9 (Pin_9), U18.12 (O4)
- new net C_D0: CNB1.1 (Pin_1), CNC1.29 (Pin_29), RN2.3 (R2), U14.18 (1Y0), U15.18 (1Y0)
- new net C_D1: CNB1.32 (Pin_32), CNC1.31 (Pin_31), RN2.5 (R4), U14.16 (1Y1), U15.16 (1Y1)
- new net C_D2: CNB1.2 (Pin_2), CNC1.2 (Pin_2), RN2.7 (R6), U14.14 (1Y2), U15.14 (1Y2)
- new net C_D3: CNB1.31 (Pin_31), CNC1.3 (Pin_3), RN2.9 (R8), U14.12 (1Y3), U15.12 (1Y3)
- new net C_D4: CNB1.3 (Pin_3), CNC1.30 (Pin_30), RN2.8 (R7), U11.3, U14.9 (2Y3), U15.9 (2Y3)
- new net C_D5: CNB1.30 (Pin_30), CNC1.4 (Pin_4), H13.5 (OUT), RN2.6 (R5), U11.6, U14.7 (2Y2), U15.7 (2Y2)
- new net C_D6: CNB1.4 (Pin_4), CNC1.5 (Pin_5), RN2.4 (R3), U11.8, U14.5 (2Y1), U15.5 (2Y1)
- new net C_D7: CNB1.29 (Pin_29), CNC1.6 (Pin_6), RN2.2 (R1), U11.11, U14.3 (2Y0), U15.3 (2Y0)
- new net C_S0: CNC1.19 (Pin_19), U18.5 (O1)
- new net C_S1: CNC1.21 (Pin_21), U18.6 (O2)
- new net C_S2: CNC1.15 (Pin_15)
- new net ENC0: AR1.5 (R4), C33.2, CN3.35 (Pin_35), SW_ENC5.1 (A), U15.2 (1A0)
- new net ENC1: AR1.4 (R3), C32.2, CN3.27 (Pin_27), SW_ENC6.1 (A), U15.4 (1A1)
- new net ENC2: AR1.6 (R5), C34.2, CN3.34 (Pin_34), SW_ENC7.1 (A), U15.6 (1A2)
- new net ENC3: AR1.8 (R7), C35.2, CN3.28 (Pin_28), SW_ENC8.1 (A), U15.8 (1A3)
- new net ENC4: AR1.9 (R8), C36.2, CN3.33 (Pin_33), SW_ENC9.1 (A), U15.11 (2A3)
- new net FS_LED: CN3.6 (Pin_6), CN_LCD1.6 (Pin_6), H12.13 (OUT)
- new net GND: C23.1, C24.2, C25.1, C26.1, C27.1, C28.1, C29.1, C30.1, C31.2, C32.1, C33.1, C34.1, C35.1, C36.1, CN3.16 (Pin_16), CN3.20 (Pin_20), CN3.22 (Pin_22), CN3.26 (Pin_26), CN3.29 (Pin_29), CN3.52 (Pin_52), CN3.59 (Pin_59), CN3.60 (Pin_60), CN5.11 (Pin_11), CN5.30 (Pin_30), CNA1.1 (Pin_1), CNA1.32 (Pin_32), CNC1.1 (Pin_1), CNC1.16 (Pin_16), CNC1.17 (Pin_17), CNC1.32 (Pin_32), CN_LCD1.13 (Pin_13), CN_LCD1.14 (Pin_14), H10.1 (GND1), H10.10 (GND6), H10.17 (GND7), H10.2 (GND2), H10.20 (GND8), H10.6 (GND3), H10.8 (GND4), H10.9 (GND5), H11.12 (GND), H12.14 (GND), H13.12 (GND), H14.5 (GND), H15.1 (Pin_1), H15.14 (Pin_14), H16.10 (GND2), H16.5 (GND1), H17.10 (GND2), H17.5 (GND1), H18.10 (GND2), H18.5 (GND1), OPT5.4, OPT6.4, OPT7.4, OPT8.4, R72.2, SW_ENC5.2 (B), SW_ENC6.2 (B), SW_ENC7.2 (B), SW_ENC8.2 (B), SW_ENC9.2 (B), U10.7 (VSS), U11.7 (GND), U12.7 (VSS), U13.16 (Vdd), U13.8 (Vss), U14.10 (GND), U15.10 (GND), U16.10 (IO), U16.4 (I7), U16.8 (GND), U17.10 (GND), U18.10 (GND)
- new net H4-3: H11.3 (IN), H11.5 (OUT), U15.17 (2A0)
- new net H4-8: H11.8 (OUT2), H17.1 (IN1)
- new net H8-4: H18.4 (IN2), U18.16 (O6)
- new net H9-11: H15.11 (Pin_11), U14.8 (1A3)
- new net H9-15: CN5.36 (Pin_36), H15.15 (Pin_15)
- new net H9-2: H15.2 (Pin_2), U10.11
- new net HOOK: AR1.2 (R1), CN5.17 (Pin_17), U11.2
- new net KBD_1: CN5.2 (Pin_2), D21.2 (A)
- new net KBD_2: CN5.1 (Pin_1), D20.2 (A)
- new net KBD_3: CN5.40 (Pin_40), CNB1.15 (Pin_15), R81.2
- new net KBD_4: CN5.39 (Pin_39), D19.2 (A)
- new net KBD_5: CN5.3 (Pin_3), CNB1.16 (Pin_16), R78.2
- new net KBD_6: CN5.38 (Pin_38), D26.2 (A)
- new net KBD_7: CN5.4 (Pin_4), CNB1.18 (Pin_18), R79.2
- new net LCD_CLK: CN3.3 (Pin_3), CNA1.10 (Pin_10), CN_LCD1.3 (Pin_3)
- new net LCD_C/~{D}: CN3.5 (Pin_5), CNA1.8 (Pin_8), CN_LCD1.5 (Pin_5)
- new net LCD_MOSI: CN3.57 (Pin_57), CNA1.24 (Pin_24), CN_LCD1.11 (Pin_11)
- new net MCU-PC0: U17.1 (OE), U18.1 (OE)
- new net PA0: CNA1.26 (Pin_26), H12.2 (IN)
- new net PA1: CNA1.7 (Pin_7), H12.8 (IN)
- new net PA2: CNA1.27 (Pin_27), H12.11 (IN)
- new net PA3: CNA1.6 (Pin_6), U12.9
- new net PA4: CNA1.28 (Pin_28), H12.4 (IN)
- new net PA6: CNA1.29 (Pin_29), U13.14 (A0)
- new net PA7: CNA1.4 (Pin_4), U13.13 (A1)
- new net PB0: CNA1.22 (Pin_22), U10.1, U10.2
- new net PB1: CNA1.11 (Pin_11), H12.6 (IN)
- new net PB2: CNA1.23 (Pin_23), H13.9 (IN)
- new net PC0: CN5.23 (Pin_23), CNA1.18 (Pin_18), U10.13, U10.6, U12.11, U12.13, U13.1 (~{EN}), U13.15 (~{EN})
- new net PC1: CN3.10 (Pin_10), CNA1.15 (Pin_15), CN_COIN1.8 (Pin_8)
- new net PC2: CNA1.19 (Pin_19), CNC1.18 (Pin_18), R74.2
- new net PC3: CNA1.14 (Pin_14), H18.1 (IN1)
- new net PC4: CNA1.20 (Pin_20), H13.10 (IN)
- new net PC5: CN5.25 (Pin_25), CNA1.13 (Pin_13), R75.2
- new net PC6: CN5.27 (Pin_27), CNA1.21 (Pin_21), R76.2
- new net PD4: CNB1.19 (Pin_19), H15.9 (Pin_9)
- new net PD5: CNB1.14 (Pin_14)
- new net PHOTO_POCKET: CN3.39 (Pin_39), H14.8 (IN), OPT7.3
- new net PHOTO_R_EXIT: CN3.45 (Pin_45), OPT5.3, R84.1, R85.2
- new net PHOTO_R_IN: CN3.32 (Pin_32), H14.1 (IN), OPT8.3
- new net PHOTO_R_IN_PWR: CN3.30 (Pin_30), CN5.24 (Pin_24), H11.13 (OUT), OPT8.2
- new net PHOTO_R_POCKET_PWR: CN3.17 (Pin_17), OPT5.2, R86.1
- new net PHOTO_SAFE: CN3.41 (Pin_41), H14.3 (IN), OPT6.3
- new net REDIAL: CN5.5 (Pin_5), H13.1 (IN)
- new net RL1-R: CN5.6 (Pin_6), H13.13 (OUT)
- new net RL1-S: CN5.37 (Pin_37), H13.11 (OUT)
- new net RL2-R: CN5.7 (Pin_7), H12.7 (OUT)
- new net RL2-S: CN5.35 (Pin_35), H12.10 (OUT)
- new net R_MOT_A: CN3.24 (Pin_24), H10.18 (MOT2), M2.1 (+)
- new net R_MOT_B: CN3.37 (Pin_37), H10.12 (MOT1), M2.2 (-)
- new net SAFE_SW1: AR1.3 (R2), CN5.19 (Pin_19), U14.11 (2A3)
- new net SAFE_SW2: AR1.7 (R6), CN5.20 (Pin_20), U15.15 (2A1)
- new net SCL-39: CN5.15 (Pin_15), CNB1.17 (Pin_17)
- new net SCL-43: CNB1.25 (Pin_25), U10.8, U10.9
- new net SCL-44: CNB1.8 (Pin_8), H10.5 (DIR)
- new net SCL-45: CNB1.26 (Pin_26), H10.3 (~{RUN}/STOP)
- new net SCL-46: CN5.14 (Pin_14), CNB1.7 (Pin_7)
- new net SCL-47: CNB1.27 (Pin_27), U17.11 (LE)
- new net SCL-50: CNB1.6 (Pin_6), U18.11 (LE)
- new net SCL-51: CNB1.28 (Pin_28), U13.2 (A0)
- new net SCL-52: CNB1.5 (Pin_5), U13.3 (A1), U13.4 (~{Q0})
- new net SOLENOID_C_PATH: CN3.19 (Pin_19), H16.9 (SOL), SOL5.1
- new net SOLENOID_C_REJ: CN3.15 (Pin_15), H17.9 (SOL), SOL4.1
- new net SOLENOID_R_POCKET: CN3.25 (Pin_25), H18.9 (SOL), SOL6.1
- new net SW1: CN3.54 (Pin_54), CNB1.13 (Pin_13), CN_LCD1.8 (Pin_8), R82.2
- new net SW2: CN3.7 (Pin_7), CNB1.20 (Pin_20), CN_LCD1.7 (Pin_7), R80.2
- new net SW_C_PATH: CN3.18 (Pin_18), H11.1 (IN), SW_C_PATH1.1 (A)
- new net SW_C_REJ: CN3.14 (Pin_14), CN_COIN1.12 (Pin_12), H11.2 (IN), SW_REJ1.1 (A)
- new net ~{IRQ}: CNA1.31 (Pin_31), U12.10
- new net ~{I_LIMIT}: CN5.26 (Pin_26), CNA1.12 (Pin_12), R77.2
- new net ~{LCD_BUSY}: CN3.56 (Pin_56), CNA1.25 (Pin_25), CN_LCD1.10 (Pin_10)
- new net ~{LCD_CS}: CN3.4 (Pin_4), CNA1.9 (Pin_9), CN_LCD1.4 (Pin_4)
- new net ~{LCD_RESET}: CN3.55 (Pin_55), CN_LCD1.9 (Pin_9), U18.19 (O7)
- new net ~{RST}: CN3.1 (Pin_1), CNA1.2 (Pin_2), CN_LCD1.1 (Pin_1)
- no-connect marks 0 -> 24
Other:
- note added: "Connectors"
- note added: "Hookswitch"
- note added: "Power"
- note added: "This solenoid opens the currently selected coin rotor pocket to dump out its contents."
- note added: "This solenoid selects whether the coin coming out from the coin rotor's pocket is directed to the coin box or to the coin return tray"
- note added: "This solenoid selects whether the coin is directed to the coin rotor (if accepted) or to the coin return tray (if rejected)"
